File: 2023l3-int.kicad_sch (KiCad schematic)
At the start: 5 parts, among them J1 0526101433, SW1 SW_DIP_x04, U1 OpenMV H7, U2 DEV-15583, U3 BNO085

Commit message: init push
Parts:
- removed SW1: SW_DIP_x04, Button_Switch_SMD:SW_DIP_SPSTx04_Slide_6.7x11.72mm_W8.61mm_P2.54mm_LowProfile, symbol Switch:SW_DIP_x04
- added D2: LED, Connector_PinHeader_2.54mm:PinHeader_1x02_P2.54mm_Vertical, symbol Device:LED
- added R1: R_Photo, Connector_PinHeader_2.54mm:PinHeader_1x02_P2.54mm_Vertical, symbol Device:R_Photo
- added R2: R, footprints:res0603, symbol Device:R
- added SW1: SW_DIP_x03, Button_Switch_SMD:SW_DIP_SPSTx03_Slide_9.78x9.8mm_W8.61mm_P2.54mm, symbol Switch:SW_DIP_x03
Connections:
- net +3V3: now also R1.1
- net +5V: now also D2.2 (A)
- net DIP1: now also SW1.3
- net DIP2: now also SW1.2
- net DIP3: now also SW1.1
- net GND: now also D2.1 (K), R2.2, SW1.4, SW1.5, SW1.6
- net DIP4 renamed LG
- net LG: now also R1.2, R2.1

Commit message: formatted sch
Parts:
- added J2: 52610-0833, 0526100833, symbol 52610-0833:52610-0833
- renumbered D2 to D?, R1 to R?, R2 to R?, SW1 to SW?, U1 to U?, U2 to U?, U3 to U?
Connections:
- net +3V3: now also J2.2 (1_2)
- net +5V: now also J2.4 (2_2)
- net GND: now also J2.14 (7_2), J2.16 (8_2)
- net ULTRA RX: now also J2.8 (4_2)
- net ULTRA TX: now also J2.6 (3_2)
- net CAM RX renamed C RX
- net CAM TX renamed C TX
- new net COM RX: J2.12 (6_2)
- new net COM TX: J2.10 (5_2)
Other:
- note added: "Camera"
- note added: "Connections"
- note added: "IMU"
- note added: "Light Gate"
- note added: "Teensy 4.0"
- moved on the sheet: D?, J1, R?, SW?, U?
