File: 2023l3-int.kicad_sch (KiCad schematic)
At the start: 9 parts, among them J1 0526101433, J2 52610-0833

Commit message: placement done
Parts:
- removed J2: 52610-0833, 0526100833, symbol 52610-0833:52610-0833
- added J2: 52610-0833, footprints:526100633, symbol 52610:52610-0633
- J1: footprint footprints:0526101433 -> footprints:526101433; symbol 0526101433:0526101433 -> 52610:52610-1433
- R2: renamed from R?; value R -> 3K24
- U?: footprint footprints:MODULE_DEV-15583 -> footprints:teensy4; symbol Teensy 4.0:DEV-15583 -> Teensy 4.0:Teensy 4.0; now left out of the parts list
- U?: footprint footprints:MODULE_4754 -> footprints:bno085
- gave numbers to parts that had none: 3
Connections:
- net +3V3: now also J2.1
- net +5V: now also J2.3
- net C RX: no longer U?.16
- net C TX: no longer U?.17
- net GND: now also J2.11, J2.9
- net ULTRA RX renamed U TX
- net U TX: now also J2.7
- net ULTRA TX renamed U RX
- net U RX: now also J2.5
- no-connect marks 23 -> 25
Other:
- moved on the sheet: J1, SW1, U?

Commit message: 🙏🙏🙏
Parts:
- removed SW1: SW_DIP_x03, Button_Switch_SMD:SW_DIP_SPSTx03_Slide_9.78x9.8mm_W8.61mm_P2.54mm, symbol Switch:SW_DIP_x03
Connections:
- net DIP1: now also U?.16 (16/A2/RX4/SCL1); no longer U?.20 (20/A6/TX5)
- net DIP2: now also U?.17 (17/A3/TX4/SDA1); no longer U?.21 (21/A7/RX5)
- net DIP3: now also U?.20 (20/A6/TX5); no longer U?.22 (22/A8)
- new net DIP4: U?.21 (21/A7/RX5)
- no-connect marks 25 -> 24
Changed lines of the file:
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@@
   (junction (at 88.9 45.72) (diameter 0) (color 0 0 0 0)
-  )
-  (junction (at 200.66 41.91) (diameter 0) (color 0 0 0 0)
-  )
-  (junction (at 200.66 39.37) (diameter 0) (color 0 0 0 0)
   )
   (junction (at 50.8 59.69) (diameter 0) (color 0 0 0 0)
@@
   (no_connect (at 58.42 88.9))
   (no_connect (at 102.87 91.44))
-  (no_connect (at 170.18 52.07))
   (no_connect (at 102.87 93.98))
   (no_connect (at 130.81 91.44))
@@
   (no_connect (at 161.29 96.52))
   (no_connect (at 161.29 88.9))
-  (no_connect (at 170.18 49.53))
   (no_connect (at 102.87 83.82))
   (no_connect (at 102.87 86.36))
+  (no_connect (at 170.18 36.83))
   (no_connect (at 170.18 31.75))
   (no_connect (at 58.42 99.06))
@@
     (stroke (width 0) (type default))
   )
-  (wire (pts (xy 200.66 41.91) (xy 200.66 44.45))
-    (stroke (width 0) (type default))
-  )
   (wire (pts (xy 41.91 54.61) (xy 50.8 54.61))
     (stroke (width 0) (type default))
@@
     (stroke (width 0) (type default))
   )
-  (wire (pts (xy 200.66 39.37) (xy 200.66 41.91))
+  (wire (pts (xy 170.18 39.37) (xy 180.34 39.37))
     (stroke (width 0) (type default))
   )
@@
     (stroke (width 0) (type default))
   )
-  (wire (pts (xy 200.66 36.83) (xy 200.66 39.37))
-    (stroke (width 0) (type default))
-  )
   (wire (pts (xy 88.9 46.99) (xy 88.9 45.72))
     (stroke (width 0) (type default))
@@
     (stroke (width 0) (type default))
   )
+  (wire (pts (xy 170.18 52.07) (xy 180.34 52.07))
+    (stroke (width 0) (type default))
+  )
   (wire (pts (xy 82.55 38.1) (xy 88.9 38.1))
     (stroke (width 0) (type default))
   )
-  (wire (pts (xy 170.18 36.83) (xy 182.88 36.83))
-    (stroke (width 0) (type default))
-  )
   (wire (pts (xy 170.18 29.21) (xy 172.72 29.21))
     (stroke (width 0) (type default))
@@
     (stroke (width 0) (type default))
   )
-  (wire (pts (xy 198.12 36.83) (xy 200.66 36.83))
-    (stroke (width 0) (type default))
-  )
   (wire (pts (xy 41.91 31.75) (xy 49.53 31.75))
     (stroke (width 0) (type default))
@@
     (stroke (width 0) (type default))
   )
-  (wire (pts (xy 198.12 41.91) (xy 200.66 41.91))
-    (stroke (width 0) (type default))
-  )
   (wire (pts (xy 170.18 54.61) (xy 179.07 54.61))
     (stroke (width 0) (type default))
   )
-  (wire (pts (xy 170.18 39.37) (xy 182.88 39.37))
-    (stroke (width 0) (type default))
-  )
   (wire (pts (xy 25.4 77.47) (xy 25.4 85.09))
     (stroke (width 0) (type default))
@@
     (stroke (width 0) (type default))
   )
+  (wire (pts (xy 170.18 49.53) (xy 180.34 49.53))
+    (stroke (width 0) (type default))
+  )
   (wire (pts (xy 128.27 44.45) (xy 137.16 44.45))
     (stroke (width 0) (type default))
@@
     (stroke (width 0) (type default))
   )
+  (wire (pts (xy 170.18 41.91) (xy 180.34 41.91))
+    (stroke (width 0) (type default))
+  )
   (wire (pts (xy 41.91 49.53) (xy 50.8 49.53))
     (stroke (width 0) (type default))
@@
     (stroke (width 0) (type default))
   )
-  (wire (pts (xy 170.18 41.91) (xy 182.88 41.91))
-    (stroke (width 0) (type default))
-  )
   (wire (pts (xy 137.16 26.67) (xy 129.54 26.67))
     (stroke (width 0) (type default))
@@
   )
   (wire (pts (xy 128.27 31.75) (xy 137.16 31.75))
-    (stroke (width 0) (type default))
-  )
-  (wire (pts (xy 198.12 39.37) (xy 200.66 39.37))
     (stroke (width 0) (type default))
   )
@@
     (effects (font (size 1.5 1.5) (thickness 0.4) bold) (justify left bottom))
   )
-  (label "DIP1" (at 171.45 41.91 0) (fields_autoplaced)
+  (label "DIP3" (at 171.45 41.91 0) (fields_autoplaced)
     (effects (font (size 1.27 1.27)) (justify left bottom))
   )
@@
     (effects (font (size 1.27 1.27)) (justify left bottom))
   )
+  (label "DIP2" (at 171.45 49.53 0) (fields_autoplaced)
+    (effects (font (size 1.27 1.27)) (justify left bottom))
+  )
   (label "BR PWM" (at 43.18 52.07 0) (fields_autoplaced)
     (effects (font (size 1.27 1.27)) (justify left bottom))
@@
     (effects (font (size 1.27 1.27)) (justify left bottom))
   )
-  (label "DIP3" (at 171.45 36.83 0) (fields_autoplaced)
-    (effects (font (size 1.27 1.27)) (justify left bottom))
-  )
   (label "FL PWM" (at 43.18 36.83 0) (fields_autoplaced)
     (effects (font (size 1.27 1.27)) (justify left bottom))
@@
     (effects (font (size 1.27 1.27)) (justify left bottom))
   )
+  (label "DIP1" (at 171.45 52.07 0) (fields_autoplaced)
+    (effects (font (size 1.27 1.27)) (justify left bottom))
+  )
   (label "U RX" (at 129.54 46.99 0) (fields_autoplaced)
     (effects (font (size 1.27 1.27)) (justify left bottom))
@@
     (effects (font (size 1.27 1.27)) (justify left bottom))
   )
-  (label "DIP2" (at 171.45 39.37 0) (fields_autoplaced)
+  (label "DIP4" (at 171.45 39.37 0) (fields_autoplaced)
     (effects (font (size 1.27 1.27)) (justify left bottom))
   )
@@
         (path "/91e7b1c2-b009-4d84-9159-ee8884a12474"
           (reference "U2") (unit 1)
-        )
-      )
-    )
-  )
-  (symbol (lib_id "Switch:SW_DIP_x03") (at 190.5 41.91 0) (unit 1)
-    (in_bom yes) (on_board yes) (dnp no) (fields_autoplaced)
-    (property "Reference" "SW1" (at 190.5 29.21 0)
-      (effects (font (size 1.27 1.27)))
-    )
-    (property "Value" "SW_DIP_x03" (at 190.5 31.75 0)
-      (effects (font (size 1.27 1.27)))
-    )
-    (property "Footprint" "Button_Switch_SMD:SW_DIP_SPSTx03_Slide_9.78x9.8mm_W8.61mm_P2.54mm" (at 190.5 41.91 0)
-      (effects (font (size 1.27 1.27)) hide)
-    )
-    (property "Datasheet" "~" (at 190.5 41.91 0)
-      (effects (font (size 1.27 1.27)) hide)
-    )
-    (pin "1")
-    (pin "2")
-    (pin "3")
-    (pin "4")
-    (pin "5")
-    (pin "6")
-    (instances
-      (project "2023l3-int"
-        (path "/91e7b1c2-b009-4d84-9159-ee8884a12474"
-          (reference "SW1") (unit 1)
         )
       )
@@
         )
       )
-    )
-  )
-  (symbol (lib_id "power:GND") (at 200.66 44.45 0) (unit 1)
-    (in_bom yes) (on_board yes) (dnp no) (fields_autoplaced)
-    (property "Reference" "#PWR0116" (at 200.66 50.8 0)
-      (effects (font (size 1.27 1.27)) hide)
-    )
-    (property "Value" "GND" (at 200.66 49.53 0)
-      (effects (font (size 1.27 1.27)))
-    )
-    (property "Footprint" "" (at 200.66 44.45 0)
-      (effects (font (size 1.27 1.27)) hide)
-    )
-    (property "Datasheet" "" (at 200.66 44.45 0)
-      (effects (font (size 1.27 1.27)) hide)
-    )
-    (pin "1")
-    (instances
-      (project "2023l3-int"
-        (path "/91e7b1c2-b009-4d84-9159-ee8884a12474"
-          (reference "#PWR0116") (unit 1)
-        )
-      )

Commit message: 3d pcb
Parts:
- added SW1: SW_DIP_x04, Button_Switch_SMD:SW_DIP_SPSTx04_Slide_6.7x11.72mm_W8.61mm_P2.54mm_LowProfile, symbol Switch:SW_DIP_x04
Connections:
- net DIP1: now also SW1.4
- net DIP2: now also SW1.3
- net DIP3: now also SW1.2
- net DIP4: now also SW1.1
- net GND: now also SW1.5, SW1.6, SW1.7, SW1.8
Other:
- moved on the sheet: U?

Commit message: e
Connections:
- net DIP1: now also U?.22 (22/A8); no longer U?.16 (16/A2/RX4/SCL1)
- net DIP2: now also U?.21 (21/A7/RX5); no longer U?.17 (17/A3/TX4/SDA1)
- net DIP4: now also U?.17 (17/A3/TX4/SDA1); no longer U?.21 (21/A7/RX5)
- no-connect marks 24 -> 23
Changed lines of the file:
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@@
   (no_connect (at 102.87 83.82))
   (no_connect (at 102.87 86.36))
-  (no_connect (at 165.1 36.83))
   (no_connect (at 165.1 31.75))
   (no_connect (at 58.42 99.06))
@@
     (stroke (width 0) (type default))
   )
+  (wire (pts (xy 124.46 99.06) (xy 130.81 99.06))
+    (stroke (width 0) (type default))
+  )
+  (wire (pts (xy 88.9 43.18) (xy 88.9 45.72))
+    (stroke (width 0) (type default))
+  )
+  (wire (pts (xy 124.46 101.6) (xy 130.81 101.6))
+    (stroke (width 0) (type default))
+  )
+  (wire (pts (xy 41.91 46.99) (xy 50.8 46.99))
+    (stroke (width 0) (type default))
+  )
+  (wire (pts (xy 82.55 45.72) (xy 88.9 45.72))
+    (stroke (width 0) (type default))
+  )
+  (wire (pts (xy 82.55 33.02) (xy 88.9 33.02))
+    (stroke (width 0) (type default))
+  )
+  (wire (pts (xy 203.2 38.1) (xy 205.74 38.1))
+    (stroke (width 0) (type default))
+  )
+  (wire (pts (xy 88.9 46.99) (xy 88.9 45.72))
+    (stroke (width 0) (type default))
+  )
+  (wire (pts (xy 41.91 41.91) (xy 50.8 41.91))
+    (stroke (width 0) (type default))
+  )
+  (wire (pts (xy 82.55 38.1) (xy 88.9 38.1))
+    (stroke (width 0) (type default))
+  )
+  (wire (pts (xy 165.1 29.21) (xy 167.64 29.21))
+    (stroke (width 0) (type default))
+  )
+  (wire (pts (xy 165.1 34.29) (xy 173.99 34.29))
+    (stroke (width 0) (type default))
+  )
+  (wire (pts (xy 203.2 45.72) (xy 205.74 45.72))
+    (stroke (width 0) (type default))
+  )
+  (wire (pts (xy 35.56 97.79) (xy 35.56 100.33))
+    (stroke (width 0) (type default))
+  )
+  (wire (pts (xy 123.19 54.61) (xy 132.08 54.61))
+    (stroke (width 0) (type default))
+  )
+  (wire (pts (xy 161.29 101.6) (xy 163.83 101.6))
+    (stroke (width 0) (type default))
+  )
+  (wire (pts (xy 165.1 41.91) (xy 175.26 41.91))
+    (stroke (width 0) (type default))
+  )
   (wire (pts (xy 165.1 39.37) (xy 175.26 39.37))
     (stroke (width 0) (type default))
   )
-  (wire (pts (xy 124.46 99.06) (xy 130.81 99.06))
-    (stroke (width 0) (type default))
-  )
-  (wire (pts (xy 88.9 43.18) (xy 88.9 45.72))
-    (stroke (width 0) (type default))
-  )
-  (wire (pts (xy 124.46 101.6) (xy 130.81 101.6))
-    (stroke (width 0) (type default))
-  )
-  (wire (pts (xy 41.91 46.99) (xy 50.8 46.99))
-    (stroke (width 0) (type default))
-  )
-  (wire (pts (xy 82.55 45.72) (xy 88.9 45.72))
-    (stroke (width 0) (type default))
-  )
-  (wire (pts (xy 82.55 33.02) (xy 88.9 33.02))
-    (stroke (width 0) (type default))
-  )
-  (wire (pts (xy 203.2 38.1) (xy 205.74 38.1))
-    (stroke (width 0) (type default))
-  )
-  (wire (pts (xy 88.9 46.99) (xy 88.9 45.72))
-    (stroke (width 0) (type default))
-  )
-  (wire (pts (xy 41.91 41.91) (xy 50.8 41.91))
-    (stroke (width 0) (type default))
-  )
-  (wire (pts (xy 165.1 52.07) (xy 175.26 52.07))
-    (stroke (width 0) (type default))
-  )
-  (wire (pts (xy 82.55 38.1) (xy 88.9 38.1))
-    (stroke (width 0) (type default))
-  )
-  (wire (pts (xy 165.1 29.21) (xy 167.64 29.21))
-    (stroke (width 0) (type default))
-  )
-  (wire (pts (xy 165.1 34.29) (xy 173.99 34.29))
-    (stroke (width 0) (type default))
-  )
-  (wire (pts (xy 203.2 45.72) (xy 205.74 45.72))
-    (stroke (width 0) (type default))
-  )
-  (wire (pts (xy 35.56 97.79) (xy 35.56 100.33))
-    (stroke (width 0) (type default))
-  )
-  (wire (pts (xy 123.19 54.61) (xy 132.08 54.61))
-    (stroke (width 0) (type default))
-  )
-  (wire (pts (xy 161.29 101.6) (xy 163.83 101.6))
-    (stroke (width 0) (type default))
-  )
   (wire (pts (xy 41.91 31.75) (xy 49.53 31.75))
     (stroke (width 0) (type default))
@@
     (stroke (width 0) (type default))
   )
+  (wire (pts (xy 165.1 49.53) (xy 175.26 49.53))
+    (stroke (width 0) (type default))
+  )
   (wire (pts (xy 203.2 43.18) (xy 205.74 43.18))
     (stroke (width 0) (type default))
@@
     (stroke (width 0) (type default))
   )
+  (wire (pts (xy 165.1 36.83) (xy 175.26 36.83))
+    (stroke (width 0) (type default))
+  )
   (wire (pts (xy 25.4 77.47) (xy 25.4 85.09))
     (stroke (width 0) (type default))
@@
     (stroke (width 0) (type default))
   )
-  (wire (pts (xy 165.1 49.53) (xy 175.26 49.53))
-    (stroke (width 0) (type default))
-  )
   (wire (pts (xy 123.19 44.45) (xy 132.08 44.45))
     (stroke (width 0) (type default))
@@
   )
   (wire (pts (xy 41.91 39.37) (xy 50.8 39.37))
-    (stroke (width 0) (type default))
-  )
-  (wire (pts (xy 165.1 41.91) (xy 175.26 41.91))
     (stroke (width 0) (type default))
   )
@@
     (effects (font (size 1.5 1.5) (thickness 0.4) bold) (justify left bottom))
   )
+  (label "L1 TX" (at 124.46 31.75 0) (fields_autoplaced)
+    (effects (font (size 1.27 1.27)) (justify left bottom))
+  )
+  (label "C TX" (at 52.07 93.98 0) (fields_autoplaced)
+    (effects (font (size 1.27 1.27)) (justify left bottom))
+  )
+  (label "U TX" (at 124.46 49.53 0) (fields_autoplaced)
+    (effects (font (size 1.27 1.27)) (justify left bottom))
+  )
+  (label "DIP4" (at 166.37 49.53 0) (fields_autoplaced)
+    (effects (font (size 1.27 1.27)) (justify left bottom))
+  )
+  (label "BR PWM" (at 124.46 54.61 0) (fields_autoplaced)
+    (effects (font (size 1.27 1.27)) (justify left bottom))
+  )
+  (label "U TX" (at 83.82 40.64 0) (fields_autoplaced)
+    (effects (font (size 1.27 1.27)) (justify left bottom))
+  )
+  (label "DIP1" (at 166.37 36.83 0) (fields_autoplaced)
+    (effects (font (size 1.27 1.27)) (justify left bottom))
+  )
+  (label "FL DIR" (at 124.46 36.83 0) (fields_autoplaced)
+    (effects (font (size 1.27 1.27)) (justify left bottom))
+  )
+  (label "DIP1" (at 182.88 45.72 0) (fields_autoplaced)
+    (effects (font (size 1.27 1.27)) (justify left bottom))
+  )
+  (label "BR DIR" (at 43.18 54.61 0) (fields_autoplaced)
+    (effects (font (size 1.27 1.27)) (justify left bottom))
+  )
+  (label "IR TX" (at 166.37 54.61 0) (fields_autoplaced)
+    (effects (font (size 1.27 1.27)) (justify left bottom))
+  )
+  (label "BL PWM" (at 43.18 46.99 0) (fields_autoplaced)
+    (effects (font (size 1.27 1.27)) (justify left bottom))
+  )
+  (label "DIP2" (at 166.37 39.37 0) (fields_autoplaced)
+    (effects (font (size 1.27 1.27)) (justify left bottom))
+  )
   (label "DIP3" (at 166.37 41.91 0) (fields_autoplaced)
     (effects (font (size 1.27 1.27)) (justify left bottom))
   )
-  (label "L1 TX" (at 124.46 31.75 0) (fields_autoplaced)
-    (effects (font (size 1.27 1.27)) (justify left bottom))
-  )
-  (label "C TX" (at 52.07 93.98 0) (fields_autoplaced)
-    (effects (font (size 1.27 1.27)) (justify left bottom))
-  )
-  (label "U TX" (at 124.46 49.53 0) (fields_autoplaced)
-    (effects (font (size 1.27 1.27)) (justify left bottom))
-  )
-  (label "BR PWM" (at 124.46 54.61 0) (fields_autoplaced)
-    (effects (font (size 1.27 1.27)) (justify left bottom))
-  )
-  (label "U TX" (at 83.82 40.64 0) (fields_autoplaced)
-    (effects (font (size 1.27 1.27)) (justify left bottom))
-  )
-  (label "FL DIR" (at 124.46 36.83 0) (fields_autoplaced)
-    (effects (font (size 1.27 1.27)) (justify left bottom))
-  )
-  (label "DIP1" (at 182.88 45.72 0) (fields_autoplaced)
-    (effects (font (size 1.27 1.27)) (justify left bottom))
-  )
-  (label "BR DIR" (at 43.18 54.61 0) (fields_autoplaced)
-    (effects (font (size 1.27 1.27)) (justify left bottom))
-  )
-  (label "IR TX" (at 166.37 54.61 0) (fields_autoplaced)
-    (effects (font (size 1.27 1.27)) (justify left bottom))
-  )
-  (label "BL PWM" (at 43.18 46.99 0) (fields_autoplaced)
-    (effects (font (size 1.27 1.27)) (justify left bottom))
-  )
-  (label "DIP2" (at 166.37 49.53 0) (fields_autoplaced)
-    (effects (font (size 1.27 1.27)) (justify left bottom))
-  )
   (label "BR PWM" (at 43.18 52.07 0) (fields_autoplaced)
     (effects (font (size 1.27 1.27)) (justify left bottom))
@@
     (effects (font (size 1.27 1.27)) (justify left bottom))
   )
-  (label "DIP1" (at 166.37 52.07 0) (fields_autoplaced)
-    (effects (font (size 1.27 1.27)) (justify left bottom))
-  )
   (label "U RX" (at 124.46 46.99 0) (fields_autoplaced)
     (effects (font (size 1.27 1.27)) (justify left bottom))
@@
     (effects (font (size 1.27 1.27)) (justify left bottom))
   )
-  (label "DIP4" (at 166.37 39.37 0) (fields_autoplaced)
-    (effects (font (size 1.27 1.27)) (justify left bottom))
-  )
