File: 2023l3-int.kicad_sch (KiCad schematic)
At the start: 9 parts, among them J1 0526101433, J2 52610-0833, SW1 SW_DIP_x04

Commit message: i wanna kill myself
Parts:
- removed J1: 0526101433, footprints:526101433, symbol 52610:52610-1433
- added J1: 0526101433, footprints:522711479, symbol 52271-1479:52271-1479
Connections:
- net +3V3: now also D1.2 (A), J1.1
- net +5V: now also J1.2; no longer D1.2 (A)
- net BL DIR: now also J1.10
- net BL PWM: now also J1.9
- net BR DIR: now also J1.12
- net BR PWM: now also J1.11
- net FL DIR: now also J1.6
- net FL PWM: now also J1.5
- net FR DIR: now also J1.8
- net FR PWM: now also J1.7
- net GND: now also J1.13, J1.14
- net L1 RX: now also J1.3
- net L1 TX: now also J1.4
Changed lines of the file:
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@@
-    )
-  )
-  (symbol (lib_id "52610:52610-1433") (at 41.91 24.13 0) (mirror y) (unit 1)
-    (in_bom yes) (on_board yes) (dnp no)
-    (property "Reference" "J1" (at 33.02 20.32 0)
-      (effects (font (size 1.27 1.27)))
-    )
-    (property "Value" "0526101433" (at 33.02 22.86 0)
-      (effects (font (size 1.27 1.27)))
-    )
-    (property "Footprint" "footprints:526101433" (at 22.86 121.59 0)
-      (effects (font (size 1.27 1.27)) (justify left top) hide)
-    )
-    (property "Datasheet" "https://www.molex.com/pdm_docs/sd/526101233_sd.pdf" (at 22.86 221.59 0)
-      (effects (font (size 1.27 1.27)) (justify left top) hide)
-    )
-    (property "Height" "6.05" (at 22.86 421.59 0)
-      (effects (font (size 1.27 1.27)) (justify left top) hide)
-    )
-    (property "Manufacturer_Name" "Molex" (at 22.86 521.59 0)
-      (effects (font (size 1.27 1.27)) (justify left top) hide)
-    )
-    (property "Manufacturer_Part_Number" "0526101433" (at 22.86 621.59 0)
-      (effects (font (size 1.27 1.27)) (justify left top) hide)
-    )
-    (property "Mouser Part Number" "N/A" (at 22.86 721.59 0)
-      (effects (font (size 1.27 1.27)) (justify left top) hide)
-    )
-    (property "Mouser Price/Stock" "https://www.mouser.com/Search/Refine.aspx?Keyword=N%2FA" (at 22.86 821.59 0)
-      (effects (font (size 1.27 1.27)) (justify left top) hide)
-    )
-    (property "Arrow Part Number" "0526101433" (at 22.86 921.59 0)
-      (effects (font (size 1.27 1.27)) (justify left top) hide)
-    )
-    (property "Arrow Price/Stock" "https://www.arrow.com/en/products/0526101433/molex" (at 22.86 1021.59 0)
-      (effects (font (size 1.27 1.27)) (justify left top) hide)
-    )
-    (pin "1")
-    (pin "10")
-    (pin "11")
-    (pin "12")
-    (pin "13")
-    (pin "14")
-    (pin "15")
-    (pin "16")
-    (pin "17")
-    (pin "18")
-    (pin "19")
-    (pin "2")
-    (pin "20")
-    (pin "21")
-    (pin "22")
-    (pin "23")
-    (pin "24")
-    (pin "25")
-    (pin "26")
-    (pin "27")
-    (pin "28")
-    (pin "3")
-    (pin "4")
-    (pin "5")
-    (pin "6")
-    (pin "7")
-    (pin "8")
-    (pin "9")
-    (instances
-      (project "2023l3-int"
-        (path "/91e7b1c2-b009-4d84-9159-ee8884a12474"
-          (reference "J1") (unit 1)
-        )
-      )
     )
   )
@@
         (path "/91e7b1c2-b009-4d84-9159-ee8884a12474"
           (reference "#PWR0104") (unit 1)
+        )
+      )
+    )
+  )
+  (symbol (lib_id "power:+3V3") (at 25.4 77.47 0) (unit 1)
+    (in_bom yes) (on_board yes) (dnp no) (fields_autoplaced)
+    (property "Reference" "#PWR010" (at 25.4 81.28 0)
+      (effects (font (size 1.27 1.27)) hide)
+    )
+    (property "Value" "+3V3" (at 25.4 72.39 0)
+      (effects (font (size 1.27 1.27)))
+    )
+    (property "Footprint" "" (at 25.4 77.47 0)
+      (effects (font (size 1.27 1.27)) hide)
+    )
+    (property "Datasheet" "" (at 25.4 77.47 0)
+      (effects (font (size 1.27 1.27)) hide)
+    )
+    (pin "1")
+    (instances
+      (project "2023l3-int"
+        (path "/91e7b1c2-b009-4d84-9159-ee8884a12474"
+          (reference "#PWR010") (unit 1)
         )
       )
@@
         (path "/91e7b1c2-b009-4d84-9159-ee8884a12474"
           (reference "J2") (unit 1)
-        )
-      )
-    )
-  )
-  (symbol (lib_id "power:+5V") (at 25.4 77.47 0) (unit 1)
-    (in_bom yes) (on_board yes) (dnp no) (fields_autoplaced)
-    (property "Reference" "#PWR0102" (at 25.4 81.28 0)
-      (effects (font (size 1.27 1.27)) hide)
-    )
-    (property "Value" "+5V" (at 25.4 72.39 0)
-      (effects (font (size 1.27 1.27)))
-    )
-    (property "Footprint" "" (at 25.4 77.47 0)
-      (effects (font (size 1.27 1.27)) hide)
-    )
-    (property "Datasheet" "" (at 25.4 77.47 0)
-      (effects (font (size 1.27 1.27)) hide)
-    )
-    (pin "1")
-    (instances
-      (project "2023l3-int"
-        (path "/91e7b1c2-b009-4d84-9159-ee8884a12474"
-          (reference "#PWR0102") (unit 1)
         )
       )
@@
         )
       )
+    )
+  )
+  (symbol (lib_id "52271-1479:52271-1479") (at 16.51 26.67 0) (unit 1)
+    (in_bom yes) (on_board yes) (dnp no)
+    (property "Reference" "J1" (at 29.21 20.32 0)
+      (effects (font (size 1.27 1.27)))
+    )
+    (property "Value" "0526101433" (at 29.21 22.86 0)
+      (effects (font (size 1.27 1.27)))
+    )
+    (property "Footprint" "footprints:522711479" (at 38.1 121.59 0)
+      (effects (font (size 1.27 1.27)) (justify left top) hide)
+    )
+    (property "Datasheet" "http://uk.rs-online.com/web/p/products/5109607" (at 38.1 221.59 0)
+      (effects (font (size 1.27 1.27)) (justify left top) hide)
+    )
+    (property "Height" "3.2" (at 38.1 421.59 0)
+      (effects (font (size 1.27 1.27)) (justify left top) hide)
+    )
+    (property "Manufacturer_Name" "Molex" (at 38.1 521.59 0)
+      (effects (font (size 1.27 1.27)) (justify left top) hide)
+    )
+    (property "Manufacturer_Part_Number" "52271-1479" (at 38.1 621.59 0)
+      (effects (font (size 1.27 1.27)) (justify left top) hide)
+    )
+    (property "Mouser Part Number" "538-52271-1479" (at 38.1 721.59 0)
+      (effects (font (size 1.27 1.27)) (justify left top) hide)
+    )
+    (property "Mouser Price/Stock" "https://www.mouser.co.uk/ProductDetail/Molex/52271-1479?qs=nP5hwMgPNFTZQPK5cfBhrw%3D%3D" (at 38.1 821.59 0)
+      (effects (font (size 1.27 1.27)) (justify left top) hide)
+    )
+    (property "Arrow Part Number" "0526101433" (at 38.1 921.59 0)
+      (effects (font (size 1.27 1.27)) (justify left top) hide)
+    )
+    (property "Arrow Price/Stock" "https://www.arrow.com/en/products/0526101433/molex" (at 38.1 1021.59 0)
+      (effects (font (size 1.27 1.27)) (justify left top) hide)
+    )
+    (pin "1")
+    (pin "10")
+    (pin "11")
+    (pin "12")
+    (pin "13")
+    (pin "14")
+    (pin "2")
+    (pin "3")
+    (pin "4")
+    (pin "5")
+    (pin "6")
+    (pin "7")
+    (pin "8")
+    (pin "9")
+    (pin "MP1")
+    (pin "MP2")
+    (instances
+      (project "2023l3-int"
+        (path "/91e7b1c2-b009-4d84-9159-ee8884a12474"
+          (reference "J1") (unit 1)
+        )
+      )

Commit message: i wanna kill myself
Connections:
- net +3V3: now also J1.14; no longer J1.1
- net +5V: now also J1.13; no longer J1.2
- net BL DIR: now also J1.5; no longer J1.10
- net BL PWM: now also J1.6; no longer J1.9
- net BR DIR: now also J1.3; no longer J1.12
- net BR PWM: now also J1.4; no longer J1.11
- net C RX: now also U?.16 (16/A2/RX4/SCL1)
- net C TX: now also U?.17 (17/A3/TX4/SDA1)
- net DIP4: now also U?.12 (12/MISO); no longer U?.17 (17/A3/TX4/SDA1)
- net FL DIR: now also J1.9; no longer J1.6
- net FL PWM: now also J1.10; no longer J1.5
- net FR DIR: now also J1.7; no longer J1.8
- net FR PWM: now also J1.8; no longer J1.7
- net GND: now also J1.1, J1.2; no longer J1.13, J1.14
- net L1 RX: now also J1.12; no longer J1.3
- net L1 TX: now also J1.11; no longer J1.4
- no-connect marks 23 -> 22

Commit message: kill me
Parts:
- added H1, H2, H3, H4, H5, H6: MountingHole_Pad, MountingHole:MountingHole_3.2mm_M3_Pad_Via, symbol Mechanical:MountingHole_Pad
Connections:
- net GND: now also H1.1, H2.1, H3.1, H4.1, H5.1, H6.1
Changed lines of the file:
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@@
   (junction (at 88.9 45.72) (diameter 0) (color 0 0 0 0)
   )
+  (junction (at 232.41 36.83) (diameter 0) (color 0 0 0 0)
+  )
   (junction (at 205.74 43.18) (diameter 0) (color 0 0 0 0)
   )
+  (junction (at 242.57 36.83) (diameter 0) (color 0 0 0 0)
+  )
+  (junction (at 237.49 36.83) (diameter 0) (color 0 0 0 0)
+  )
   (junction (at 205.74 45.72) (diameter 0) (color 0 0 0 0)
+  )
+  (junction (at 227.33 36.83) (diameter 0) (color 0 0 0 0)
+  )
+  (junction (at 234.95 36.83) (diameter 0) (color 0 0 0 0)
   )
   (junction (at 205.74 40.64) (diameter 0) (color 0 0 0 0)
@@
   (no_connect (at 130.81 93.98))
   (no_connect (at 161.29 91.44))
+  (wire (pts (xy 222.25 35.56) (xy 222.25 36.83))
+    (stroke (width 0) (type default))
+  )
   (wire (pts (xy 123.19 36.83) (xy 132.08 36.83))
     (stroke (width 0) (type default))
@@
     (stroke (width 0) (type default))
   )
+  (wire (pts (xy 232.41 35.56) (xy 232.41 36.83))
+    (stroke (width 0) (type default))
+  )
   (wire (pts (xy 165.1 57.15) (xy 173.99 57.15))
     (stroke (width 0) (type default))
@@
     (stroke (width 0) (type default))
   )
+  (wire (pts (xy 227.33 36.83) (xy 232.41 36.83))
+    (stroke (width 0) (type default))
+  )
   (wire (pts (xy 35.56 87.63) (xy 35.56 88.9))
     (stroke (width 0) (type default))
@@
     (stroke (width 0) (type default))
   )
+  (wire (pts (xy 227.33 35.56) (xy 227.33 36.83))
+    (stroke (width 0) (type default))
+  )
   (wire (pts (xy 88.9 43.18) (xy 88.9 45.72))
     (stroke (width 0) (type default))
   )
+  (wire (pts (xy 232.41 36.83) (xy 234.95 36.83))
+    (stroke (width 0) (type default))
+  )
   (wire (pts (xy 124.46 101.6) (xy 130.81 101.6))
     (stroke (width 0) (type default))
@@
     (stroke (width 0) (type default))
   )
+  (wire (pts (xy 237.49 35.56) (xy 237.49 36.83))
+    (stroke (width 0) (type default))
+  )
   (wire (pts (xy 88.9 46.99) (xy 88.9 45.72))
     (stroke (width 0) (type default))
@@
     (stroke (width 0) (type default))
   )
+  (wire (pts (xy 222.25 36.83) (xy 227.33 36.83))
+    (stroke (width 0) (type default))
+  )
   (wire (pts (xy 165.1 39.37) (xy 175.26 39.37))
     (stroke (width 0) (type default))
@@
     (stroke (width 0) (type default))
   )
+  (wire (pts (xy 234.95 36.83) (xy 237.49 36.83))
+    (stroke (width 0) (type default))
+  )
   (wire (pts (xy 203.2 43.18) (xy 205.74 43.18))
     (stroke (width 0) (type default))
@@
     (stroke (width 0) (type default))
   )
+  (wire (pts (xy 237.49 36.83) (xy 242.57 36.83))
+    (stroke (width 0) (type default))
+  )
   (wire (pts (xy 205.74 43.18) (xy 205.74 45.72))
     (stroke (width 0) (type default))
@@
     (stroke (width 0) (type default))
   )
+  (wire (pts (xy 247.65 36.83) (xy 247.65 35.56))
+    (stroke (width 0) (type default))
+  )
   (wire (pts (xy 132.08 26.67) (xy 124.46 26.67))
     (stroke (width 0) (type default))
@@
   )
   (wire (pts (xy 123.19 49.53) (xy 132.08 49.53))
+    (stroke (width 0) (type default))
+  )
+  (wire (pts (xy 242.57 35.56) (xy 242.57 36.83))
+    (stroke (width 0) (type default))
+  )
+  (wire (pts (xy 242.57 36.83) (xy 247.65 36.83))
+    (stroke (width 0) (type default))
+  )
+  (wire (pts (xy 234.95 36.83) (xy 234.95 39.37))
     (stroke (width 0) (type default))
   )
@@
   (label "SCL" (at 125.73 99.06 0) (fields_autoplaced)
     (effects (font (size 1.27 1.27)) (justify left bottom))
+  )
+  (symbol (lib_id "Mechanical:MountingHole_Pad") (at 242.57 33.02 0) (unit 1)
+    (in_bom yes) (on_board yes) (dnp no) (fields_autoplaced)
+    (property "Reference" "H5" (at 245.11 31.115 0)
+      (effects (font (size 1.27 1.27)) (justify left))
+    )
+    (property "Value" "MountingHole_Pad" (at 245.11 33.655 0)
+      (effects (font (size 1.27 1.27)) (justify left))
+    )
+    (property "Footprint" "MountingHole:MountingHole_3.2mm_M3_Pad_Via" (at 242.57 33.02 0)
+      (effects (font (size 1.27 1.27)) hide)
+    )
+    (property "Datasheet" "~" (at 242.57 33.02 0)
+      (effects (font (size 1.27 1.27)) hide)
+    )
+    (pin "1")
+    (instances
+      (project "2023l3-int"
+        (path "/91e7b1c2-b009-4d84-9159-ee8884a12474"
+          (reference "H5") (unit 1)
+        )
+      )
+    )
   )
   (symbol (lib_id "Device:R_Photo") (at 35.56 83.82 0) (unit 1)
@@
     )
   )
+  (symbol (lib_id "Mechanical:MountingHole_Pad") (at 222.25 33.02 0) (unit 1)
+    (in_bom yes) (on_board yes) (dnp no) (fields_autoplaced)
+    (property "Reference" "H1" (at 224.79 31.115 0)
+      (effects (font (size 1.27 1.27)) (justify left))
+    )
+    (property "Value" "MountingHole_Pad" (at 224.79 33.655 0)
+      (effects (font (size 1.27 1.27)) (justify left))
+    )
+    (property "Footprint" "MountingHole:MountingHole_3.2mm_M3_Pad_Via" (at 222.25 33.02 0)
+      (effects (font (size 1.27 1.27)) hide)
+    )
+    (property "Datasheet" "~" (at 222.25 33.02 0)
+      (effects (font (size 1.27 1.27)) hide)
+    )
+    (pin "1")
+    (instances
+      (project "2023l3-int"
+        (path "/91e7b1c2-b009-4d84-9159-ee8884a12474"
+          (reference "H1") (unit 1)
+        )
+      )
+    )
+  )
+  (symbol (lib_id "Mechanical:MountingHole_Pad") (at 237.49 33.02 0) (unit 1)
+    (in_bom yes) (on_board yes) (dnp no) (fields_autoplaced)
+    (property "Reference" "H4" (at 240.03 31.115 0)
+      (effects (font (size 1.27 1.27)) (justify left))
+    )
+    (property "Value" "MountingHole_Pad" (at 240.03 33.655 0)
+      (effects (font (size 1.27 1.27)) (justify left))
+    )
+    (property "Footprint" "MountingHole:MountingHole_3.2mm_M3_Pad_Via" (at 237.49 33.02 0)
+      (effects (font (size 1.27 1.27)) hide)
+    )
+    (property "Datasheet" "~" (at 237.49 33.02 0)
+      (effects (font (size 1.27 1.27)) hide)
+    )
+    (pin "1")
+    (instances
+      (project "2023l3-int"
+        (path "/91e7b1c2-b009-4d84-9159-ee8884a12474"
+          (reference "H4") (unit 1)
+        )
+      )
+    )
+  )
   (symbol (lib_id "power:+5V") (at 88.9 35.56 270) (unit 1)
     (in_bom yes) (on_board yes) (dnp no) (fields_autoplaced)
@@
     )
   )
+  (symbol (lib_id "power:GND") (at 234.95 39.37 0) (unit 1)
+    (in_bom yes) (on_board yes) (dnp no) (fields_autoplaced)
+    (property "Reference" "#PWR011" (at 234.95 45.72 0)
+      (effects (font (size 1.27 1.27)) hide)
+    )
+    (property "Value" "GND" (at 234.95 44.45 0)
+      (effects (font (size 1.27 1.27)))
+    )
+    (property "Footprint" "" (at 234.95 39.37 0)
+      (effects (font (size 1.27 1.27)) hide)
+    )
+    (property "Datasheet" "" (at 234.95 39.37 0)
+      (effects (font (size 1.27 1.27)) hide)
+    )
+    (pin "1")
+    (instances
+      (project "2023l3-int"
+        (path "/91e7b1c2-b009-4d84-9159-ee8884a12474"
+          (reference "#PWR011") (unit 1)
+        )
+      )
+    )
+  )
   (symbol (lib_id "power:GND") (at 88.9 46.99 0) (unit 1)
     (in_bom yes) (on_board yes) (dnp no) (fields_autoplaced)
@@
         (path "/91e7b1c2-b009-4d84-9159-ee8884a12474"
           (reference "#PWR02") (unit 1)
+        )
+      )
+    )
+  )
+  (symbol (lib_id "Mechanical:MountingHole_Pad") (at 247.65 33.02 0) (unit 1)
+    (in_bom yes) (on_board yes) (dnp no) (fields_autoplaced)
+    (property "Reference" "H6" (at 250.19 31.115 0)
+      (effects (font (size 1.27 1.27)) (justify left))
+    )
+    (property "Value" "MountingHole_Pad" (at 250.19 33.655 0)
+      (effects (font (size 1.27 1.27)) (justify left))
+    )
+    (property "Footprint" "MountingHole:MountingHole_3.2mm_M3_Pad_Via" (at 247.65 33.02 0)
+      (effects (font (size 1.27 1.27)) hide)
+    )
+    (property "Datasheet" "~" (at 247.65 33.02 0)
+      (effects (font (size 1.27 1.27)) hide)
+    )
+    (pin "1")
+    (instances
+      (project "2023l3-int"
+        (path "/91e7b1c2-b009-4d84-9159-ee8884a12474"
+          (reference "H6") (unit 1)
         )
       )
@@
         (path "/91e7b1c2-b009-4d84-9159-ee8884a12474"
           (reference "D1") (unit 1)
+        )
+      )
+    )
+  )
+  (symbol (lib_id "Mechanical:MountingHole_Pad") (at 227.33 33.02 0) (unit 1)
+    (in_bom yes) (on_board yes) (dnp no) (fields_autoplaced)
+    (property "Reference" "H2" (at 229.87 31.115 0)
+      (effects (font (size 1.27 1.27)) (justify left))
+    )
+    (property "Value" "MountingHole_Pad" (at 229.87 33.655 0)
+      (effects (font (size 1.27 1.27)) (justify left))
+    )
+    (property "Footprint" "MountingHole:MountingHole_3.2mm_M3_Pad_Via" (at 227.33 33.02 0)
+      (effects (font (size 1.27 1.27)) hide)
+    )
+    (property "Datasheet" "~" (at 227.33 33.02 0)
+      (effects (font (size 1.27 1.27)) hide)
+    )
+    (pin "1")
+    (instances
+      (project "2023l3-int"
+        (path "/91e7b1c2-b009-4d84-9159-ee8884a12474"
+          (reference "H2") (unit 1)
         )
       )
@@
         )
       )
+    )
+  )
+  (symbol (lib_id "Mechanical:MountingHole_Pad") (at 232.41 33.02 0) (unit 1)
+    (in_bom yes) (on_board yes) (dnp no) (fields_autoplaced)
+    (property "Reference" "H3" (at 234.95 31.115 0)
+      (effects (font (size 1.27 1.27)) (justify left))
+    )
+    (property "Value" "MountingHole_Pad" (at 234.95 33.655 0)
+      (effects (font (size 1.27 1.27)) (justify left))
+    )
+    (property "Footprint" "MountingHole:MountingHole_3.2mm_M3_Pad_Via" (at 232.41 33.02 0)
+      (effects (font (size 1.27 1.27)) hide)
+    )
+    (property "Datasheet" "~" (at 232.41 33.02 0)
+      (effects (font (size 1.27 1.27)) hide)
+    )
+    (pin "1")
+    (instances
+      (project "2023l3-int"
+        (path "/91e7b1c2-b009-4d84-9159-ee8884a12474"
+          (reference "H3") (unit 1)
+        )
+      )

Commit message: kill me
Parts:
- removed J2: 52610-0833, footprints:526100633, symbol 52610:52610-0633
- added U28: Seeed Studio XIAO ESP32C3, footprints:XIAO-ESP32C3-THT, symbol Seeed_Studio_XIAO_Series:Seeed_Studio_XIAO_ESP32C3
Connections:
- net +5V: now also U28.13 (5V)
- net GND: now also U28.12 (GND)
- net U RX renamed BT RX
- net BT RX: now also U28.6 (TX)
- net U TX renamed BT TX
- net BT TX: now also U28.7 (RX)
- no-connect marks 22 -> 32
Other:
- note added: "ESP32-C3"
- moved on the sheet: J1
