File: 2023l3-int.kicad_sch (KiCad schematic)
At the start: 15 parts, among them J1 0526101433, SW1 SW_DIP_x04, U28 Seeed Studio XIAO ESP32C3

Commit message: kms
Parts:
- removed D1: LED, Connector_PinHeader_2.54mm:PinHeader_1x02_P2.54mm_Vertical, symbol Device:LED
- removed H5, H6: MountingHole_Pad, MountingHole:MountingHole_3.2mm_M3_Pad_Via, symbol Mechanical:MountingHole_Pad
- removed R1: R_Photo, Connector_PinHeader_2.54mm:PinHeader_1x02_P2.54mm_Vertical, symbol Device:R_Photo
- removed R2: 3K24, footprints:res0603, symbol Device:R
- added R1: 3K24, footprints:res0603, symbol Device:R
Connections:
- net +3V3: now also J1.1; no longer J1.14
- net +5V: now also J1.2; no longer J1.13
- net BL DIR: now also J1.10, U?.7 (7/RX2); no longer J1.5, U?.9
- net BL PWM: now also J1.9; no longer J1.6
- net BR DIR: now also J1.12, U?.9; no longer J1.3, U?.11 (11/MOSI)
- net BR PWM: now also J1.11, U?.8 (8/TX2); no longer J1.4, U?.10 (10/CS)
- net BT RX: now also U?.21 (21/A7/RX5); no longer U?.7 (7/RX2)
- net BT TX: now also U?.20 (20/A6/TX5); no longer U?.8 (8/TX2)
- net DIP2: now also U?.12 (12/MISO); no longer U?.21 (21/A7/RX5)
- net DIP3: now also U?.11 (11/MOSI); no longer U?.20 (20/A6/TX5)
- net DIP4: now also U?.10 (10/CS); no longer U?.12 (12/MISO)
- net FL DIR: now also J1.6; no longer J1.9
- net FL PWM: now also J1.5; no longer J1.10
- net FR DIR: now also J1.8; no longer J1.7
- net FR PWM: now also J1.7; no longer J1.8
- net GND: now also J1.13, J1.14, R1.1; no longer J1.1, J1.2
- net L1 RX: now also J1.3; no longer J1.12
- net L1 TX: now also J1.4; no longer J1.11
- net LG: now also R1.2
Other:
- note removed: "Light Gate"
- moved on the sheet: SW1, U?

Commit message: oui oui
Parts:
- removed R1: 3K24, footprints:res0603, symbol Device:R
- removed U28: Seeed Studio XIAO ESP32C3, footprints:XIAO-ESP32C3-THT, symbol Seeed_Studio_XIAO_Series:Seeed_Studio_XIAO_ESP32C3
- added U28: xiao-esp32c3, footprints:xiao-esp32c3, symbol Seeed_Studio_XIAO_Series:xiao-esp32c3
Connections:
- net +5V: now also U28.13 (5V)
- net BT RX: now also U28.6 (TX)
- net BT TX: now also U28.7 (RX)
- net GND: now also U28.12 (GND)
- net L1 RX: now also J1.4; no longer J1.3
- net L1 TX: now also J1.3; no longer J1.4

Commit message: reee
Connections:
- net +3V3: now also U?.JP1_1 (VIN)
- net +5V: no longer U?.JP1_1 (VIN)
- net L1 RX: now also J1.3; no longer J1.4
- net L1 TX: now also J1.4; no longer J1.3
Changed lines of the file:
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@@
     (effects (font (size 1.27 1.27)) (justify left bottom))
   )
-  (label "L1 RX" (at 44.45 33.02 0) (fields_autoplaced)
+  (label "L1 RX" (at 44.45 30.48 0) (fields_autoplaced)
     (effects (font (size 1.27 1.27)) (justify left bottom))
   )
@@
   )
   (label "DIP3" (at 124.46 57.15 0) (fields_autoplaced)
+    (effects (font (size 1.27 1.27)) (justify left bottom))
+  )
+  (label "L1 TX" (at 44.45 33.02 0) (fields_autoplaced)
     (effects (font (size 1.27 1.27)) (justify left bottom))
   )
@@
   (label "BT TX" (at 102.87 52.07 180) (fields_autoplaced)
     (effects (font (size 1.27 1.27)) (justify right bottom))
-  )
-  (label "L1 TX" (at 44.45 30.48 0) (fields_autoplaced)
-    (effects (font (size 1.27 1.27)) (justify left bottom))
   )
   (label "BT RX" (at 171.45 39.37 180) (fields_autoplaced)
@@
     )
   )
-  (symbol (lib_id "power:+5V") (at 95.25 83.82 90) (mirror x) (unit 1)
-    (in_bom yes) (on_board yes) (dnp no) (fields_autoplaced)
-    (property "Reference" "#PWR?" (at 99.06 83.82 0)
-      (effects (font (size 1.27 1.27)) hide)
-    )
-    (property "Value" "+5V" (at 91.44 83.82 90)
-      (effects (font (size 1.27 1.27)) (justify left))
-    )
-    (property "Footprint" "" (at 95.25 83.82 0)
-      (effects (font (size 1.27 1.27)) hide)
-    )
-    (property "Datasheet" "" (at 95.25 83.82 0)
-      (effects (font (size 1.27 1.27)) hide)
-    )
-    (pin "1")
-    (instances
-      (project "2024l3"
-        (path "/03701560-9a76-47ab-9e75-66b9cf21bc38"
-          (reference "#PWR?") (unit 1)
-        )
-      )
-      (project "2024l1"
-        (path "/5be543b5-1bdc-438f-a916-f916127c0a2b"
-          (reference "#PWR?") (unit 1)
-        )
-      )
-      (project "2023l3-int"
-        (path "/91e7b1c2-b009-4d84-9159-ee8884a12474"
-          (reference "#PWR07") (unit 1)
-        )
-      )
-    )
-  )
   (symbol (lib_id "power:GND") (at 100.33 39.37 90) (unit 1)
     (in_bom yes) (on_board yes) (dnp no) (fields_autoplaced)
@@
         )
       )
+    )
+  )
+  (symbol (lib_id "power:+3V3") (at 95.25 83.82 90) (unit 1)
+    (in_bom yes) (on_board yes) (dnp no) (fields_autoplaced)
+    (property "Reference" "#PWR06" (at 99.06 83.82 0)
+      (effects (font (size 1.27 1.27)) hide)
+    )
+    (property "Value" "+3V3" (at 91.44 84.455 90)
+      (effects (font (size 1.27 1.27)) (justify left))
+    )
+    (property "Footprint" "" (at 95.25 83.82 0)
+      (effects (font (size 1.27 1.27)) hide)
+    )
+    (property "Datasheet" "" (at 95.25 83.82 0)
+      (effects (font (size 1.27 1.27)) hide)
+    )
+    (pin "1")
+    (instances
+      (project "2023l3-int"
+        (path "/91e7b1c2-b009-4d84-9159-ee8884a12474"
+          (reference "#PWR06") (unit 1)
+        )
+      )

Commit message: done
Connections:
- net C RX: now also U?.15 (15/A1/RX3); no longer U?.16 (16/A2/RX4/SCL1)
- net C TX: now also U?.14 (14/A0/TX3); no longer U?.17 (17/A3/TX4/SDA1)
- net IR RX: now also U?.17 (17/A3/TX4/SDA1); no longer U?.14 (14/A0/TX3)
- net IR TX: now also U?.16 (16/A2/RX4/SCL1); no longer U?.15 (15/A1/RX3)
Other:
- moved on the sheet: SW1
Changed lines of the file:
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@@
   (junction (at 232.41 36.83) (diameter 0) (color 0 0 0 0)
   )
-  (junction (at 205.74 52.07) (diameter 0) (color 0 0 0 0)
-  )
-  (junction (at 205.74 54.61) (diameter 0) (color 0 0 0 0)
+  (junction (at 205.74 41.91) (diameter 0) (color 0 0 0 0)
+  )
+  (junction (at 205.74 44.45) (diameter 0) (color 0 0 0 0)
   )
   (junction (at 227.33 36.83) (diameter 0) (color 0 0 0 0)
@@
   (junction (at 234.95 36.83) (diameter 0) (color 0 0 0 0)
   )
-  (junction (at 205.74 49.53) (diameter 0) (color 0 0 0 0)
+  (junction (at 205.74 39.37) (diameter 0) (color 0 0 0 0)
   )
   (junction (at 52.07 58.42) (diameter 0) (color 0 0 0 0)
@@
     (stroke (width 0) (type default))
   )
-  (wire (pts (xy 205.74 54.61) (xy 205.74 58.42))
-    (stroke (width 0) (type default))
-  )
-  (wire (pts (xy 205.74 49.53) (xy 205.74 52.07))
+  (wire (pts (xy 205.74 44.45) (xy 205.74 48.26))
+    (stroke (width 0) (type default))
+  )
+  (wire (pts (xy 205.74 39.37) (xy 205.74 41.91))
     (stroke (width 0) (type default))
   )
@@
     (stroke (width 0) (type default))
   )
-  (wire (pts (xy 165.1 57.15) (xy 173.99 57.15))
-    (stroke (width 0) (type default))
-  )
   (wire (pts (xy 43.18 58.42) (xy 52.07 58.42))
     (stroke (width 0) (type default))
@@
     (stroke (width 0) (type default))
   )
+  (wire (pts (xy 165.1 52.07) (xy 173.99 52.07))
+    (stroke (width 0) (type default))
+  )
   (wire (pts (xy 43.18 53.34) (xy 52.07 53.34))
     (stroke (width 0) (type default))
@@
     (stroke (width 0) (type default))
   )
-  (wire (pts (xy 165.1 49.53) (xy 175.26 49.53))
-    (stroke (width 0) (type default))
-  )
-  (wire (pts (xy 203.2 46.99) (xy 205.74 46.99))
+  (wire (pts (xy 203.2 36.83) (xy 205.74 36.83))
     (stroke (width 0) (type default))
   )
@@
     (stroke (width 0) (type default))
   )
-  (wire (pts (xy 203.2 54.61) (xy 205.74 54.61))
+  (wire (pts (xy 203.2 44.45) (xy 205.74 44.45))
     (stroke (width 0) (type default))
   )
@@
     (stroke (width 0) (type default))
   )
-  (wire (pts (xy 165.1 52.07) (xy 175.26 52.07))
-    (stroke (width 0) (type default))
-  )
   (wire (pts (xy 123.19 49.53) (xy 132.08 49.53))
     (stroke (width 0) (type default))
@@
     (stroke (width 0) (type default))
   )
-  (wire (pts (xy 203.2 52.07) (xy 205.74 52.07))
+  (wire (pts (xy 203.2 41.91) (xy 205.74 41.91))
     (stroke (width 0) (type default))
   )
@@
     (stroke (width 0) (type default))
   )
-  (wire (pts (xy 181.61 52.07) (xy 187.96 52.07))
+  (wire (pts (xy 181.61 41.91) (xy 187.96 41.91))
+    (stroke (width 0) (type default))
+  )
+  (wire (pts (xy 165.1 49.53) (xy 173.99 49.53))
     (stroke (width 0) (type default))
   )
@@
     (stroke (width 0) (type default))
   )
-  (wire (pts (xy 165.1 54.61) (xy 173.99 54.61))
-    (stroke (width 0) (type default))
-  )
-  (wire (pts (xy 205.74 46.99) (xy 205.74 49.53))
+  (wire (pts (xy 205.74 36.83) (xy 205.74 39.37))
     (stroke (width 0) (type default))
   )
@@
     (stroke (width 0) (type default))
   )
-  (wire (pts (xy 181.61 49.53) (xy 187.96 49.53))
-    (stroke (width 0) (type default))
-  )
-  (wire (pts (xy 203.2 49.53) (xy 205.74 49.53))
+  (wire (pts (xy 181.61 39.37) (xy 187.96 39.37))
+    (stroke (width 0) (type default))
+  )
+  (wire (pts (xy 203.2 39.37) (xy 205.74 39.37))
     (stroke (width 0) (type default))
   )
@@
     (stroke (width 0) (type default))
   )
+  (wire (pts (xy 165.1 54.61) (xy 175.26 54.61))
+    (stroke (width 0) (type default))
+  )
   (wire (pts (xy 95.25 36.83) (xy 100.33 36.83))
     (stroke (width 0) (type default))
@@
     (stroke (width 0) (type default))
   )
-  (wire (pts (xy 181.61 46.99) (xy 187.96 46.99))
+  (wire (pts (xy 181.61 36.83) (xy 187.96 36.83))
     (stroke (width 0) (type default))
   )
@@
     (stroke (width 0) (type default))
   )
-  (wire (pts (xy 205.74 52.07) (xy 205.74 54.61))
+  (wire (pts (xy 205.74 41.91) (xy 205.74 44.45))
     (stroke (width 0) (type default))
   )
@@
     (stroke (width 0) (type default))
   )
+  (wire (pts (xy 165.1 57.15) (xy 175.26 57.15))
+    (stroke (width 0) (type default))
+  )
   (wire (pts (xy 74.93 92.71) (xy 74.93 96.52))
     (stroke (width 0) (type default))
   )
-  (wire (pts (xy 181.61 54.61) (xy 187.96 54.61))
+  (wire (pts (xy 181.61 44.45) (xy 187.96 44.45))
     (stroke (width 0) (type default))
   )
@@
     (effects (font (size 1.27 1.27)) (justify left bottom))
   )
-  (label "C RX" (at 166.37 52.07 0) (fields_autoplaced)
+  (label "C RX" (at 166.37 54.61 0) (fields_autoplaced)
     (effects (font (size 1.27 1.27)) (justify left bottom))
   )
@@
     (effects (font (size 1.27 1.27)) (justify left bottom))
   )
-  (label "DIP1" (at 182.88 54.61 0) (fields_autoplaced)
+  (label "DIP1" (at 182.88 44.45 0) (fields_autoplaced)
     (effects (font (size 1.27 1.27)) (justify left bottom))
   )
@@
     (effects (font (size 1.27 1.27)) (justify left bottom))
   )
-  (label "IR TX" (at 166.37 54.61 0) (fields_autoplaced)
-    (effects (font (size 1.27 1.27)) (justify left bottom))
-  )
   (label "BL PWM" (at 44.45 45.72 0) (fields_autoplaced)
     (effects (font (size 1.27 1.27)) (justify left bottom))
@@
     (effects (font (size 1.27 1.27)) (justify left bottom))
   )
-  (label "IR RX" (at 166.37 57.15 0) (fields_autoplaced)
-    (effects (font (size 1.27 1.27)) (justify left bottom))
-  )
   (label "BT RX" (at 69.85 52.07 0) (fields_autoplaced)
     (effects (font (size 1.27 1.27)) (justify left bottom))
@@
     (effects (font (size 1.27 1.27)) (justify left bottom))
   )
+  (label "IR TX" (at 166.37 52.07 0) (fields_autoplaced)
+    (effects (font (size 1.27 1.27)) (justify left bottom))
+  )
   (label "SCL" (at 166.37 44.45 0) (fields_autoplaced)
     (effects (font (size 1.27 1.27)) (justify left bottom))
   )
-  (label "DIP3" (at 182.88 49.53 0) (fields_autoplaced)
-    (effects (font (size 1.27 1.27)) (justify left bottom))
-  )
-  (label "DIP2" (at 182.88 52.07 0) (fields_autoplaced)
+  (label "C TX" (at 166.37 57.15 0) (fields_autoplaced)
+    (effects (font (size 1.27 1.27)) (justify left bottom))
+  )
+  (label "DIP3" (at 182.88 39.37 0) (fields_autoplaced)
+    (effects (font (size 1.27 1.27)) (justify left bottom))
+  )
+  (label "DIP2" (at 182.88 41.91 0) (fields_autoplaced)
     (effects (font (size 1.27 1.27)) (justify left bottom))
   )
@@
     (effects (font (size 1.27 1.27)) (justify left bottom))
   )
-  (label "C TX" (at 166.37 49.53 0) (fields_autoplaced)
-    (effects (font (size 1.27 1.27)) (justify left bottom))
-  )
   (label "SDA" (at 92.71 101.6 0) (fields_autoplaced)
     (effects (font (size 1.27 1.27)) (justify left bottom))
@@
     (effects (font (size 1.27 1.27)) (justify left bottom))
   )
-  (label "DIP4" (at 182.88 46.99 0) (fields_autoplaced)
+  (label "DIP4" (at 182.88 36.83 0) (fields_autoplaced)
     (effects (font (size 1.27 1.27)) (justify left bottom))
   )
@@
     (effects (font (size 1.27 1.27)) (justify right bottom))
   )
+  (label "IR RX" (at 166.37 49.53 0) (fields_autoplaced)
+    (effects (font (size 1.27 1.27)) (justify left bottom))
+  )
   (label "BT RX" (at 171.45 39.37 180) (fields_autoplaced)
     (effects (font (size 1.27 1.27)) (justify right bottom))
+  )
+  (global_label "IR TX" (shape bidirectional) (at 173.99 52.07 0)
+    (effects (font (size 1.27 1.27)) (justify left))
+    (property "Intersheetrefs" "${INTERSHEET_REFS}" (at 182.4983 52.07 0)
+      (effects (font (size 1.27 1.27)) hide)
+    )
+  )
+  (global_label "IR RX" (shape bidirectional) (at 173.99 49.53 0)
+    (effects (font (size 1.27 1.27)) (justify left))
+    (property "Intersheetrefs" "${INTERSHEET_REFS}" (at 182.4983 49.53 0)
+      (effects (font (size 1.27 1.27)) hide)
+    )
   )
   (symbol (lib_id "OpenMV:OpenMV_H7") (at 48.26 78.74 0) (unit 1)
@@
     )
   )
-  (symbol (lib_id "power:GND") (at 205.74 58.42 0) (unit 1)
+  (symbol (lib_id "power:GND") (at 205.74 48.26 0) (unit 1)
     (in_bom yes) (on_board yes) (dnp no) (fields_autoplaced)
-    (property "Reference" "#PWR09" (at 205.74 64.77 0)
-      (effects (font (size 1.27 1.27)) hide)
-    )
-    (property "Value" "GND" (at 205.74 63.5 0)
-      (effects (font (size 1.27 1.27)))
-    )
-    (property "Footprint" "" (at 205.74 58.42 0)
-      (effects (font (size 1.27 1.27)) hide)
-    )
-    (property "Datasheet" "" (at 205.74 58.42 0)
+    (property "Reference" "#PWR09" (at 205.74 54.61 0)
+      (effects (font (size 1.27 1.27)) hide)
+    )
+    (property "Value" "GND" (at 205.74 53.34 0)
+      (effects (font (size 1.27 1.27)))
+    )
+    (property "Footprint" "" (at 205.74 48.26 0)
+      (effects (font (size 1.27 1.27)) hide)
+    )
+    (property "Datasheet" "" (at 205.74 48.26 0)
       (effects (font (size 1.27 1.27)) hide)
     )
@@
     )
   )
-  (symbol (lib_id "Switch:SW_DIP_x04") (at 195.58 52.07 0) (unit 1)
+  (symbol (lib_id "Switch:SW_DIP_x04") (at 195.58 41.91 0) (unit 1)
     (in_bom yes) (on_board yes) (dnp no) (fields_autoplaced)
-    (property "Reference" "SW1" (at 195.58 40.64 0)
-      (effects (font (size 1.27 1.27)))
-    )
-    (property "Value" "SW_DIP_x04" (at 195.58 43.18 0)
-      (effects (font (size 1.27 1.27)))
-    )
-    (property "Footprint" "Button_Switch_SMD:SW_DIP_SPSTx04_Slide_6.7x11.72mm_W8.61mm_P2.54mm_LowProfile" (at 195.58 52.07 0)
-      (effects (font (size 1.27 1.27)) hide)
-    )
-    (property "Datasheet" "~" (at 195.58 52.07 0)
-      (effects (font (size 1.27 1.27)) hide)
-    )
+    (property "Reference" "SW1" (at 195.58 30.48 0)
+      (effects (font (size 1.27 1.27)))
+    )
+    (property "Value" "SW_DIP_x04" (at 195.58 33.02 0)
+      (effects (font (size 1.27 1.27)))
+    )
+    (property "Footprint" "Button_Switch_SMD:SW_DIP_SPSTx04_Slide_6.7x11.72mm_W8.61mm_P2.54mm_LowProfile" (at 195.58 41.91 0)
+      (effects (font (size 1.27 1.27)) hide)
+    )
+    (property "Datasheet" "~" (at 195.58 41.91 0)
+      (effects (font (size 1.27 1.27)) hide)
+    )

Commit message: silkscreen
Parts:
- removed SW1: SW_DIP_x04, Button_Switch_SMD:SW_DIP_SPSTx04_Slide_6.7x11.72mm_W8.61mm_P2.54mm_LowProfile, symbol Switch:SW_DIP_x04
- added J2: Conn_01x03_Pin, Connector_PinHeader_2.54mm:PinHeader_1x03_P2.54mm_Vertical, symbol Connector:Conn_01x03_Pin
- added R?: 10K, footprints:res0603, symbol Device:R
- added R?: 1K, footprints:res0603, symbol Device:R
- added SW1: SW_DIP_x02, Button_Switch_SMD:SW_DIP_SPSTx02_Slide_6.7x6.64mm_W8.61mm_P2.54mm_LowProfile, symbol Switch:SW_DIP_x02
- added SW?: SW_Push, footprints:SW_PUSH_SPST, symbol Switch:SW_Push
Connections:
- net DIP3 is gone; now on net DIP2: U?.11 (11/MOSI)
- net +3V3: now also R?.1
- net DIP1: now also U?.12 (12/MISO), SW1.2; no longer U?.22 (22/A8)
- net DIP2: now also SW1.1; no longer U?.12 (12/MISO)
- net GND: now also J2.3 (Pin_3), R?.2, SW1.3, SW1.4
- net DIP4 renamed ESC
- net ESC: now also J2.1 (Pin_1)
- new net: R?.1, SW?.1
- new net T_RST: R?.2, SW?.2, U?.22 (22/A8)
- no-connect marks 32 -> 33

Commit message: final
Connections:
- net GND: now also J1.MP1, J1.MP2
Other:
- moved on the sheet: J1
