File: 2023l3-int.kicad_sch (KiCad schematic)
At the start: 14 parts, among them J1 0526101433, J2 Conn_01x03_Pin, SW1 SW_DIP_x02, U28 xiao-esp32c3

Commit message: jlcpcb
Connections:
- net GND: no longer H1.1, H2.1, H3.1, H4.1
- no-connect marks 33 -> 37
Changed lines of the file:
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@@
 (kicad_sch (version 20230121) (generator eeschema)
   (paper "A4")
-  (junction (at 232.41 36.83) (diameter 0) (color 0 0 0 0)
-  )
   (junction (at 19.05 27.94) (diameter 0) (color 0 0 0 0)
   )
@@
   (junction (at 168.91 90.17) (diameter 0) (color 0 0 0 0)
   )
-  (junction (at 227.33 36.83) (diameter 0) (color 0 0 0 0)
-  )
-  (junction (at 234.95 36.83) (diameter 0) (color 0 0 0 0)
-  )
   (junction (at 53.34 58.42) (diameter 0) (color 0 0 0 0)
   )
+  (no_connect (at 227.33 35.56))
   (no_connect (at 97.79 96.52))
   (no_connect (at 25.4 88.9))
@@
   (no_connect (at 25.4 96.52))
   (no_connect (at 77.47 39.37))
+  (no_connect (at 232.41 35.56))
   (no_connect (at 77.47 44.45))
   (no_connect (at 128.27 96.52))
@@
   (no_connect (at 165.1 59.69))
   (no_connect (at 25.4 83.82))
+  (no_connect (at 237.49 35.56))
   (no_connect (at 25.4 86.36))
   (no_connect (at 128.27 83.82))
   (no_connect (at 95.25 41.91))
+  (no_connect (at 222.25 35.56))
   (no_connect (at 25.4 81.28))
   (no_connect (at 97.79 93.98))
@@
   (no_connect (at 190.5 91.44))
   (no_connect (at 77.47 46.99))
-  (wire (pts (xy 222.25 35.56) (xy 222.25 36.83))
-    (stroke (width 0) (type default))
-  )
   (wire (pts (xy 123.19 36.83) (xy 132.08 36.83))
     (stroke (width 0) (type default))
@@
     (stroke (width 0) (type default))
   )
-  (wire (pts (xy 232.41 35.56) (xy 232.41 36.83))
-    (stroke (width 0) (type default))
-  )
   (wire (pts (xy 44.45 58.42) (xy 53.34 58.42))
     (stroke (width 0) (type default))
@@
     (stroke (width 0) (type default))
   )
-  (wire (pts (xy 227.33 36.83) (xy 232.41 36.83))
-    (stroke (width 0) (type default))
-  )
   (wire (pts (xy 74.93 99.06) (xy 74.93 102.87))
     (stroke (width 0) (type default))
@@
     (stroke (width 0) (type default))
   )
-  (wire (pts (xy 227.33 35.56) (xy 227.33 36.83))
-    (stroke (width 0) (type default))
-  )
-  (wire (pts (xy 232.41 36.83) (xy 234.95 36.83))
-    (stroke (width 0) (type default))
-  )
   (wire (pts (xy 91.44 101.6) (xy 97.79 101.6))
     (stroke (width 0) (type default))
@@
     (stroke (width 0) (type default))
   )
-  (wire (pts (xy 237.49 35.56) (xy 237.49 36.83))
-    (stroke (width 0) (type default))
-  )
   (wire (pts (xy 44.45 40.64) (xy 53.34 40.64))
     (stroke (width 0) (type default))
@@
     (stroke (width 0) (type default))
   )
-  (wire (pts (xy 222.25 36.83) (xy 227.33 36.83))
-    (stroke (width 0) (type default))
-  )
   (wire (pts (xy 168.91 90.17) (xy 158.75 90.17))
     (stroke (width 0) (type default))
@@
     (stroke (width 0) (type default))
   )
-  (wire (pts (xy 234.95 36.83) (xy 237.49 36.83))
-    (stroke (width 0) (type default))
-  )
   (wire (pts (xy 168.91 113.03) (xy 168.91 115.57))
     (stroke (width 0) (type default))
@@
   )
   (wire (pts (xy 104.14 52.07) (xy 95.25 52.07))
-    (stroke (width 0) (type default))
-  )
-  (wire (pts (xy 234.95 36.83) (xy 234.95 39.37))
     (stroke (width 0) (type default))
   )
@@
         )
       )
-      (project "2023l3-int-rounded"
+      (project "2023l3-int"
         (path "/91e7b1c2-b009-4d84-9159-ee8884a12474"
           (reference "U2") (unit 1)
@@
     (pin "MP2")
     (instances
-      (project "2023l3-int-rounded"
+      (project "2023l3-int"
         (path "/91e7b1c2-b009-4d84-9159-ee8884a12474"
           (reference "J1") (unit 1)
@@
     (pin "1")
     (instances
-      (project "2023l3-int-rounded"
+      (project "2023l3-int"
         (path "/91e7b1c2-b009-4d84-9159-ee8884a12474"
           (reference "#PWR09") (unit 1)
@@
         )
       )
-      (project "2023l3-int-rounded"
+      (project "2023l3-int"
         (path "/91e7b1c2-b009-4d84-9159-ee8884a12474/b6f041e8-1c4e-4d5e-bf26-3f97c4703dae"
           (reference "R3") (unit 1)
@@
         )
       )
-      (project "2023l3-int-rounded"
+      (project "2023l3-int"
         (path "/91e7b1c2-b009-4d84-9159-ee8884a12474"
           (reference "#PWR0118") (unit 1)
@@
     (pin "1")
     (instances
-      (project "2023l3-int-rounded"
+      (project "2023l3-int"
         (path "/91e7b1c2-b009-4d84-9159-ee8884a12474"
           (reference "#PWR0104") (unit 1)
@@
         )
       )
-      (project "2023l3-int-rounded"
+      (project "2023l3-int"
         (path "/91e7b1c2-b009-4d84-9159-ee8884a12474"
           (reference "#PWR03") (unit 1)
@@
         )
       )
-      (project "2023l3-int-rounded"
+      (project "2023l3-int"
         (path "/91e7b1c2-b009-4d84-9159-ee8884a12474"
           (reference "#PWR014") (unit 1)
@@
         )
       )
-      (project "2023l3-int-rounded"
+      (project "2023l3-int"
         (path "/91e7b1c2-b009-4d84-9159-ee8884a12474"
           (reference "U1") (unit 1)
@@
     (pin "1")
     (instances
-      (project "2023l3-int-rounded"
+      (project "2023l3-int"
         (path "/91e7b1c2-b009-4d84-9159-ee8884a12474"
           (reference "#PWR0105") (unit 1)
@@
         )
       )
-      (project "2023l3-int-rounded"
+      (project "2023l3-int"
         (path "/91e7b1c2-b009-4d84-9159-ee8884a12474/b6f041e8-1c4e-4d5e-bf26-3f97c4703dae"
           (reference "R5") (unit 1)
@@
         )
       )
-      (project "2023l3-int-rounded"
+      (project "2023l3-int"
         (path "/91e7b1c2-b009-4d84-9159-ee8884a12474/b6f041e8-1c4e-4d5e-bf26-3f97c4703dae"
           (reference "#PWR0167") (unit 1)
@@
     (pin "1")
     (instances
-      (project "2023l3-int-rounded"
+      (project "2023l3-int"
         (path "/91e7b1c2-b009-4d84-9159-ee8884a12474"
           (reference "#PWR05") (unit 1)
@@
     (pin "3")
     (instances
-      (project "2023l3-int-rounded"
+      (project "2023l3-int"
         (path "/91e7b1c2-b009-4d84-9159-ee8884a12474"
           (reference "J2") (unit 1)
@@
     (pin "1")
     (instances
-      (project "2023l3-int-rounded"
+      (project "2023l3-int"
         (path "/91e7b1c2-b009-4d84-9159-ee8884a12474"
           (reference "H1") (unit 1)
@@
     (pin "1")
     (instances
-      (project "2023l3-int-rounded"
+      (project "2023l3-int"
         (path "/91e7b1c2-b009-4d84-9159-ee8884a12474"
           (reference "H4") (unit 1)
@@
         )
       )
-      (project "2023l3-int-rounded"
+      (project "2023l3-int"
         (path "/91e7b1c2-b009-4d84-9159-ee8884a12474"
           (reference "#PWR04") (unit 1)
@@
     (pin "1")
     (instances
-      (project "2023l3-int-rounded"
+      (project "2023l3-int"
         (path "/91e7b1c2-b009-4d84-9159-ee8884a12474"
           (reference "#PWR06") (unit 1)
-        )
-      )
-    )
-  )
-  (symbol (lib_id "power:GND") (at 234.95 39.37 0) (unit 1)
-    (in_bom yes) (on_board yes) (dnp no) (fields_autoplaced)
-    (property "Reference" "#PWR011" (at 234.95 45.72 0)
-      (effects (font (size 1.27 1.27)) hide)
-    )
-    (property "Value" "GND" (at 234.95 44.45 0)
-      (effects (font (size 1.27 1.27)))
-    )
-    (property "Footprint" "" (at 234.95 39.37 0)
-      (effects (font (size 1.27 1.27)) hide)
-    )
-    (property "Datasheet" "" (at 234.95 39.37 0)
-      (effects (font (size 1.27 1.27)) hide)
-    )
-    (pin "1")
-    (instances
-      (project "2023l3-int-rounded"
-        (path "/91e7b1c2-b009-4d84-9159-ee8884a12474"
-          (reference "#PWR011") (unit 1)
         )
       )
@@
     (pin "4")
     (instances
-      (project "2023l3-int-rounded"
+      (project "2023l3-int"
         (path "/91e7b1c2-b009-4d84-9159-ee8884a12474"
           (reference "SW1") (unit 1)
@@
     (pin "1")
     (instances
-      (project "2023l3-int-rounded"
+      (project "2023l3-int"
         (path "/91e7b1c2-b009-4d84-9159-ee8884a12474"
           (reference "#PWR01") (unit 1)
@@
         )
       )
-      (project "2023l3-int-rounded"
+      (project "2023l3-int"
         (path "/91e7b1c2-b009-4d84-9159-ee8884a12474"
           (reference "#PWR02") (unit 1)
@@
         )
       )
-      (project "2023l3-int-rounded"
+      (project "2023l3-int"
         (path "/91e7b1c2-b009-4d84-9159-ee8884a12474"
           (reference "#PWR08") (unit 1)
@@
     (pin "1")
     (instances
-      (project "2023l3-int-rounded"
+      (project "2023l3-int"
         (path "/91e7b1c2-b009-4d84-9159-ee8884a12474"
           (reference "H2") (unit 1)
@@
         )
       )
-      (project "2023l3-int-rounded"
+      (project "2023l3-int"
         (path "/91e7b1c2-b009-4d84-9159-ee8884a12474/b6f041e8-1c4e-4d5e-bf26-3f97c4703dae"
           (reference "SW2") (unit 1)
@@
         )
       )
-      (project "2023l3-int-rounded"
+      (project "2023l3-int"
         (path "/91e7b1c2-b009-4d84-9159-ee8884a12474"
           (reference "#PWR0117") (unit 1)
@@
         )
       )
-      (project "2023l3-int-rounded"
+      (project "2023l3-int"
         (path "/91e7b1c2-b009-4d84-9159-ee8884a12474"
           (reference "U3") (unit 1)
@@
         )
       )
-      (project "2023l3-int-rounded"
+      (project "2023l3-int"
         (path "/91e7b1c2-b009-4d84-9159-ee8884a12474"
           (reference "#PWR0115") (unit 1)
@@
     (pin "9")
     (instances
-      (project "2023l3-int-rounded"
+      (project "2023l3-int"
         (path "/91e7b1c2-b009-4d84-9159-ee8884a12474"
           (reference "U28") (unit 1)
@@
         )
       )
-      (project "2023l3-int-rounded"
+      (project "2023l3-int"
         (path "/91e7b1c2-b009-4d84-9159-ee8884a12474/b6f041e8-1c4e-4d5e-bf26-3f97c4703dae"
           (reference "#PWR0171") (unit 1)
@@
     (pin "1")
     (instances
-      (project "2023l3-int-rounded"
+      (project "2023l3-int"
         (path "/91e7b1c2-b009-4d84-9159-ee8884a12474"
           (reference "H3") (unit 1)
@@
     )
     (instances
-      (project "2023l3-int-rounded"
+      (project "2023l3-int"
         (path "/91e7b1c2-b009-4d84-9159-ee8884a12474" (page "3"))
       )
