File: 2023l3-int.kicad_pcb (KiCad board)
At the start: 2 copper layers, 180.2 x 155.6 mm, 53 parts, among them IC1 STM32F103CBTx, J1 0526101433, J2 52610-0833, J3 Conn_01x04, SW1 SW_DIP_x04, SW2 SW_Push, U1 DEV-15583, U10 TSSP58038, U11 TSSP58038, U12 TSSP58038, U13 TSSP58038, U14 TSSP58038, U15 TSSP58038, U16 TSSP58038, U17 TSSP58038, U18 TSSP58038, U19 TSSP58038, U2 OpenMV H7, U20 TSSP58038, U21 TSSP58038, U22 TSSP58038, U23 TSSP58038, U24 TSSP58038, U25 TSSP58038, U26 TSSP58038, U27 TSSP58038, U3 BNO085, U4 TSSP58038, U5 TSSP58038, U6 TSSP58038, U7 TSSP58038, U8 TSSP58038, U9 TSSP58038, Y1 8Mhz

Commit message: kill me
Parts:
- moved J2 1.00 mm to (204.6, 100.0)
Routing:
- net /U TX: track 20.1 -> 19.1 mm
- net /U RX: track 19.4 -> 18.4 mm
Other:
- board text added: "BL DIR"
- board text added: "BL PWM"
- board text added: "BR DIR"
- board text added: "BR PWM"
- board text added: "FL DIR"
- board text added: "FL PWM"
- board text added: "FR DIR"
- board text added: "FR PWM"
- board text removed: "SWCLK"
- board text removed: "SWDIO"

Commit message: kill me
Parts:
- removed J2: 52610-0833, footprints:526100633
- added U28: Seeed Studio XIAO ESP32C3, footprints:XIAO-ESP32C3-THT, F.Cu at (160.0, 72.0)
Connections:
- U1 pad 7: /U RX -> /BT RX
- U1 pad 8: /U TX -> /BT TX
Routing:
- net /U TX: track 19.1 -> 0.00 mm
- net /U RX: track 18.4 -> 0.00 mm
- net +3V3: track 619.7 -> 603.4 mm
- net +5V: track 113.6 -> 105.8 mm, vias 1 -> 0
- net /IR/IR12: track 61.5 -> 64.1 mm

Commit message: kms
Parts:
- removed D1: LED, Connector_PinHeader_2.54mm:PinHeader_1x02_P2.54mm_Vertical
- removed the H1 at (111.6, 188.2)
- removed the H2 at (208.4, 188.2)
- removed R2: 3K24, footprints:res0603
- J1: moved to F.Cu
- R1: value R_Photo -> 3K24; footprint Connector_PinHeader_2.54mm:PinHeader_1x02_P2.54mm_Vertical -> footprints:res0603; moved to F.Cu
- moved R1 90.1 mm to (174.9, 110.2), turned to 90 degrees
- moved U3 61.0 mm to (160.0, 69.5), turned to 0 degrees
- moved U28 56.0 mm to (160.0, 128.0)
- moved J1 29.1 mm to (196.9, 100.0), turned to 90 degrees
- moved U4 9.61 mm to (160.0, 147.0), turned to 0 degrees
- moved U16 9.61 mm to (160.0, 53.0), turned to 180 degrees
- moved U10 9.61 mm to (207.0, 100.0), turned to 90 degrees
- moved U22 9.61 mm to (113.0, 100.0), turned to -90 degrees
- moved U26 9.61 mm to (136.5, 140.7), turned to -30 degrees
- moved U8 9.61 mm to (200.7, 123.5), turned to 60 degrees
- moved U20 9.61 mm to (119.3, 76.5), turned to -120 degrees
- moved U14 9.61 mm to (183.5, 59.3), turned to 150 degrees
- moved U24 9.61 mm to (119.3, 123.5), turned to -60 degrees
- moved U6 9.61 mm to (183.5, 140.7), turned to 30 degrees
- moved U12 9.61 mm to (200.7, 76.5), turned to 120 degrees
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- renumbered H3 to H1, H4 to H2, H6 to H3, H5 to H4
Connections:
- J1 pad 1: GND -> +3V3
- J1 pad 10: /FL PWM -> /BL DIR
- J1 pad 11: /L1 TX -> /BR PWM
- J1 pad 12: /L1 RX -> /BR DIR
- J1 pad 13: +5V -> GND
- J1 pad 14: +3V3 -> GND
- J1 pad 2: GND -> +5V
- J1 pad 3: /BR DIR -> /L1 RX
- J1 pad 4: /BR PWM -> /L1 TX
- J1 pad 5: /BL DIR -> /FL PWM
- J1 pad 6: /BL PWM -> /FL DIR
- J1 pad 7: /FR DIR -> /FR PWM
- J1 pad 8: /FR PWM -> /FR DIR
- J1 pad 9: /FL DIR -> /BL PWM
- R1 pad 1: +3V3 -> GND
- U1 pad 10: /BR PWM -> /DIP4
- U1 pad 11: /BR DIR -> /DIP3
- U1 pad 12: /DIP4 -> /DIP2
- U1 pad 20: /DIP3 -> /BT TX
- U1 pad 21: /DIP2 -> /BT RX
- U1 pad 7: /BT RX -> /BL DIR
- U1 pad 8: /BT TX -> /BR PWM
- U1 pad 9: /BL DIR -> /BR DIR
Routing:
- net +3V3: track 603.4 -> 19.3 mm, vias 3 -> 1
- net /LG: track 120.4 -> 0.00 mm, vias 2 -> 0
- net /IR/IR6: track 83.3 -> 0.00 mm
- net /IR/IR7: track 78.0 -> 0.00 mm
- net /IR/IR5: track 73.0 -> 0.00 mm
- net /IR/IR3: track 68.7 -> 0.00 mm
- net /IR/IR12: track 64.1 -> 0.00 mm
- net /IR/IR4: track 63.2 -> 0.00 mm
- net /IR/IR2: track 61.5 -> 0.00 mm
- net /IR/IR16: track 60.6 -> 0.00 mm
- net /IR/IR1: track 60.4 -> 0.00 mm
- net /IR/IR13: track 59.4 -> 0.00 mm
- net /IR/IR19: track 55.8 -> 0.00 mm
- net /IR/IR20: track 55.3 -> 0.00 mm
- net /IR/IR14: track 54.5 -> 0.00 mm
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Other:
- board size 180.2 x 155.6 mm -> 180.2 x 110 mm
- board text added: "Robotics"
- board text added: "Sentinels"
- board text added: "Singapore"
- board text added: "Team"
- board text removed: "KEEP HANDS OFF"

Commit message: oui oui
Parts:
- removed R1: 3K24, footprints:res0603
- U28: value Seeed Studio XIAO ESP32C3 -> xiao-esp32c3; footprint footprints:XIAO-ESP32C3-THT -> footprints:xiao-esp32c3
- moved R5 2.13 mm to (140.8, 106.8)
- moved SW2 2.13 mm to (145.0, 106.8)
- moved R3 2.13 mm to (149.2, 106.8)
- moved R4 0.89 mm to (150.8, 97.8)
- moved C3 0.60 mm to (163.6, 92.4)
- moved C4 0.60 mm to (152.4, 96.4)
- moved C1 0.36 mm to (167.6, 103.6)
- moved U1 0.18 mm to (180.5, 100.0)
- moved D2 0.10 mm to (152.4, 104.3)
Connections:
- J1 pad 3: /L1 RX -> /L1 TX
- J1 pad 4: /L1 TX -> /L1 RX
Routing:
- net +5V: track 136.5 -> 47.7 mm
- net /IR/IR7: track 0.00 -> 68.3 mm
- net /IR/IR6: track 0.00 -> 62.2 mm
- net /IR/IR8: track 0.00 -> 59.4 mm
- net /IR/IR5: track 0.00 -> 52.9 mm
- net /IR/IR4: track 0.00 -> 51.3 mm
- net /IR/IR9: track 0.00 -> 51.1 mm
- net /IR/IR13: track 0.00 -> 50.0 mm
- net /IR/IR12: track 0.00 -> 49.8 mm
- net /IR/IR10: track 0.00 -> 48.2 mm
- net /IR/IR3: track 0.00 -> 47.7 mm
- net /IR/IR21: track 0.00 -> 47.6 mm
- net /IR/IR17: track 0.00 -> 47.4 mm
- net /IR/IR24: track 0.00 -> 47.3 mm
- net /IR/IR20: track 0.00 -> 46.6 mm
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Other:
- outline, holes or cut-outs redrawn

Commit message: reee
Routing:
- net +3V3: track 3.61 -> 70.4 mm, vias 0 -> 2
- net +5V: track 47.7 -> 93.2 mm, vias 0 -> 2
- net /BT RX: track 0.00 -> 36.4 mm
- net /SCL: track 0.00 -> 32.7 mm
- net /BT TX: track 0.00 -> 28.1 mm
- net /SDA: track 0.00 -> 25.7 mm
- net /IR/SWDIO: track 0.00 -> 24.2 mm, vias 0 -> 1
- net /IR/SWCLK: track 0.00 -> 15.4 mm, vias 0 -> 1
- net /IR/RST: track 0.00 -> 11.8 mm
- net Net-(R5-Pad1): track 0.00 -> 2.52 mm
- net /IR/IR7: track 68.3 -> 69.7 mm
- net /IR/IR14: track 45.4 -> 46.7 mm

Commit message: reee
Parts:
- moved C6 7.67 mm to (158.5, 107.2), turned to -135 degrees
- moved Y1 7.57 mm to (155.4, 104.1)
- moved C5 7.43 mm to (152.4, 100.9), turned to -135 degrees
- moved R4 5.56 mm to (148.0, 93.0), turned to 0 degrees
- moved C4 2.72 mm to (151.6, 99.0), turned to 180 degrees
- moved J1 0.72 mm to (197.6, 100.0)
Connections:
- IC1 pad 21: /IR/IR7 -> unconnected-(IC1-PB10-Pad21)
- IC1 pad 27: unconnected-(IC1-PB14-Pad27) -> /IR/IR7
- J1 pad 3: /L1 TX -> /L1 RX
- J1 pad 4: /L1 RX -> /L1 TX
- U3 pad JP1_1: +5V -> +3V3
Routing:
- net +3V3: track 70.4 -> 159.9 mm, vias 2 -> 4
- net /IR/IR5: track 52.9 -> 76.9 mm
- net /IR/IR6: track 62.2 -> 85.9 mm
- net /IR/IR12: track 49.8 -> 70.4 mm
- net /IR/IR13: track 50.0 -> 66.2 mm
- net /IR/IR4: track 51.3 -> 66.9 mm
- net +5V: track 93.2 -> 78.5 mm, vias 2 -> 1
- net /IR/IR3: track 47.7 -> 60.2 mm
- net /IR/IR14: track 46.7 -> 58.8 mm
- net Net-(IC1-PD1): track 0.00 -> 12.1 mm, vias 0 -> 1
- net Net-(IC1-PD0): track 0.00 -> 9.74 mm, vias 0 -> 1
- net /IR/BOOT: track 0.00 -> 9.63 mm
- net /IR/IR1: track 45.2 -> 54.3 mm
- net /IR/IR16: track 43.8 -> 52.5 mm
- net /L1 RX: track 20.2 -> 12.2 mm
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
Commit message: reee
Routing:
- net +3V3: track 159.9 -> 464.9 mm
- net /IR/SWCLK: track 15.2 -> 21.6 mm
- net /IR/IR13: track 66.2 -> 72.0 mm
- net /IR/IR7: track 68.8 -> 73.8 mm
- net /IR/IR14: track 58.8 -> 63.6 mm
- net /IR/IR12: track 70.4 -> 74.8 mm
- net /IR/IR17: track 49.3 -> 50.6 mm
- net /IR/IR5: track 76.9 -> 77.8 mm
- net Net-(IC1-PD1): track 12.1 -> 13.0 mm
- net /IR/IR20: track 47.8 -> 48.6 mm
- net /IR/BOOT: track 9.63 -> 10.4 mm
- net /IR/IR15: track 52.2 -> 53.0 mm
- net /IR/IR23: track 45.6 -> 46.3 mm
- net Net-(IC1-PD0): track 9.74 -> 10.4 mm
- net /IR/IR22: track 46.2 -> 46.8 mm

Commit message: done
Parts:
- J3: footprint Connector_PinHeader_2.54mm:PinHeader_1x04_P2.54mm_Horizontal -> Connector_JST:JST_SH_SM04B-SRSS-TB_1x04-1MP_P1.00mm_Horizontal
- moved J3 26.3 mm to (126.6, 100.0), turned to -90 degrees
- moved U28 2.00 mm to (160.0, 130.0), turned to 180 degrees
Connections:
- IC1 pad 27: /IR/IR7 -> /IR/IR8
- IC1 pad 28: /IR/IR8 -> /IR/IR7
- IC1 pad 30: /IR/IR RX -> IR RX
- IC1 pad 31: /IR/IR TX -> IR TX
- J3 pad 1: +3V3 -> GND
- J3 pad 2: /IR/SWCLK -> /IR/SWDIO
- J3 pad 3: /IR/SWDIO -> /IR/SWCLK
- J3 pad 4: GND -> +3V3
- U1 pad 14: /IR RX -> /C TX
- U1 pad 15: /IR TX -> /C RX
- U1 pad 16: /C RX -> IR TX
- U1 pad 17: /C TX -> IR RX
Routing:
- net /IR/IR5: track 77.8 -> 51.9 mm
- net /IR/IR6: track 85.9 -> 60.4 mm
- net /IR/SWDIO: track 17.4 -> 41.2 mm, vias 0 -> 2
- net +5V: track 78.5 -> 100.4 mm
- net IR TX: track 0.00 -> 16.4 mm, vias 0 -> 1
- net IR RX: track 0.00 -> 15.1 mm, vias 0 -> 1
- net /IR/SWCLK: track 21.6 -> 36.5 mm, vias 0 -> 2
- net /IR/IR3: track 60.2 -> 46.3 mm
- net /IR/IR4: track 66.9 -> 53.4 mm
- net /BT RX: track 34.0 -> 20.7 mm
- net /BT TX: track 21.3 -> 29.6 mm
- net /IR/IR1: track 54.3 -> 46.0 mm
- net /IR/IR2: track 53.1 -> 46.6 mm
- net /IR/IR8: track 63.0 -> 57.1 mm
- net /IR/IR14: track 63.6 -> 58.2 mm
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