File: 2023l3-int.kicad_pcb (KiCad board)
At the start: 2 copper layers, 180.2 x 110 mm, 48 parts, among them IC1 STM32F103CBTx, J1 0526101433, J3 Conn_01x04, SW1 SW_DIP_x04, SW2 SW_Push, U1 DEV-15583, U10 TSSP58038, U11 TSSP58038, U12 TSSP58038, U13 TSSP58038, U14 TSSP58038, U15 TSSP58038, U16 TSSP58038, U17 TSSP58038, U18 TSSP58038, U19 TSSP58038, U2 OpenMV H7, U20 TSSP58038, U21 TSSP58038, U22 TSSP58038, U23 TSSP58038, U24 TSSP58038, U25 TSSP58038, U26 TSSP58038, U27 TSSP58038, U28 xiao-esp32c3, U3 BNO085, U4 TSSP58038, U5 TSSP58038, U6 TSSP58038, U7 TSSP58038, U8 TSSP58038, U9 TSSP58038, Y1 8Mhz

Commit message: silkscreen
Parts:
- added J2: Conn_01x03_Pin, Connector_PinHeader_2.54mm:PinHeader_1x03_P2.54mm_Vertical, F.Cu at (186.6, 122.0)
- added R1: 10K, footprints:res0603, F.Cu at (175.0, 121.6)
- added R2: 1K, footprints:res0603, F.Cu at (175.0, 129.6)
- added SW3: SW_Push, footprints:SW_PUSH_SPST, F.Cu at (175.0, 125.6)
- SW1: value SW_DIP_x04 -> SW_DIP_x02; footprint Button_Switch_SMD:SW_DIP_SPSTx04_Slide_6.7x11.72mm_W8.61mm_P2.54mm_LowProfile -> Button_Switch_SMD:SW_DIP_SPSTx02_Slide_6.7x6.64mm_W8.61mm_P2.54mm_LowProfile
- moved SW1 0.89 mm to (180.8, 125.6)
Connections:
- SW1 pad 1: /DIP4 -> /DIP2
- SW1 pad 2: /DIP3 -> /DIP1
- SW1 pad 3: /DIP2 -> GND
- SW1 pad 4: /DIP1 -> GND
- U1 pad 10: /DIP4 -> /ESC
- U1 pad 11: /DIP3 -> /DIP2
- U1 pad 12: /DIP2 -> /DIP1
- U1 pad 22: /DIP1 -> /T_RST
Routing:
- net /DIP3: track 37.1 -> 0.00 mm
- net /ESC: track 0.00 -> 34.8 mm
- net /DIP4: track 33.5 -> 0.00 mm
- net +3V3: track 466.3 -> 495.2 mm, vias 5 -> 6
- net /DIP1: track 15.7 -> 41.4 mm
- net /T_RST: track 0.00 -> 18.1 mm
- net /DIP2: track 40.7 -> 37.8 mm
- net Net-(R2-Pad1): track 0.00 -> 2.32 mm
- net /IR/IR6: track 60.4 -> 62.4 mm
- net /IR/IR5: track 51.9 -> 53.6 mm
Other:
- board text added: "Goal"
- board text added: "PWM"
- board text added: "Playstyle"
- board text added: "T RST"

Commit message: drc errors
Routing:
- net /IR/SWDIO: track 41.2 -> 48.9 mm
- net +3V3: track 495.2 -> 495.9 mm
Changed lines of the file:
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@@
   (segment (start 195.154 106.5) (end 192.725 106.5) (width 0.254) (layer "F.Cu") (net 3))
   (segment (start 149.225 107.575) (end 151 107.575) (width 0.254) (layer "F.Cu") (net 3))
-  (segment (start 151.067052 107.575) (end 152.807737 105.834315) (width 0.254) (layer "F.Cu") (net 3))
+  (segment (start 154.33137 105) (end 155.165685 105.834315) (width 0.254) (layer "F.Cu") (net 3))
+  (segment (start 153.642052 105) (end 154.33137 105) (width 0.254) (layer "F.Cu") (net 3))
   (segment (start 168.4 101.6) (end 168.4 101.66863) (width 0.254) (layer "F.Cu") (net 3))
   (segment (start 175.774999 121.575) (end 175.774999 119.625001) (width 0.25) (layer "F.Cu") (net 3))
@@
   (segment (start 152.401212 99.001212) (end 152.4 99) (width 0.254) (layer "F.Cu") (net 3))
   (segment (start 128.6 101.5) (end 125.1 101.5) (width 0.254) (layer "F.Cu") (net 3))
-  (segment (start 151 107.575) (end 151.067052 107.575) (width 0.254) (layer "F.Cu") (net 3))
   (segment (start 164.887876 100.998788) (end 164.998788 100.998788) (width 0.254) (layer "F.Cu") (net 3))
   (segment (start 125.1 101.5) (end 124.2 100.6) (width 0.254) (layer "F.Cu") (net 3))
+  (segment (start 151 107.575) (end 151.067052 107.575) (width 0.254) (layer "F.Cu") (net 3))
   (segment (start 160.8 94.913336) (end 160.998788 95.112124) (width 0.254) (layer "F.Cu") (net 3))
   (segment (start 206.0559 109.711048) (end 204.166948 111.6) (width 0.254) (layer "F.Cu") (net 3))
   (segment (start 160.8 93.8) (end 160.8 94.913336) (width 0.254) (layer "F.Cu") (net 3))
-  (segment (start 152.807737 105.834315) (end 155.165685 105.834315) (width 0.254) (layer "F.Cu") (net 3))
+  (segment (start 151.067052 107.575) (end 153.642052 105) (width 0.254) (layer "F.Cu") (net 3))
   (via (at 168.4 101.6) (size 0.8) (drill 0.4) (layers "F.Cu" "B.Cu") (net 3))
   (via (at 151 107.575) (size 0.8) (drill 0.4) (layers "F.Cu" "B.Cu") (net 3))
@@
   (segment (start 195.030051 126.970652) (end 195.030051 131.437949) (width 0.254) (layer "B.Cu") (net 3))
   (segment (start 181.300295 58.0268) (end 173.793748 58.0268) (width 0.254) (layer "B.Cu") (net 3))
+  (segment (start 175.774999 119.625001) (end 176.149998 120) (width 0.25) (layer "B.Cu") (net 3))
   (segment (start 157.46 53) (end 159.3041 54.8441) (width 0.254) (layer "B.Cu") (net 3))
   (segment (start 153.225 109.8) (end 160.2 109.8) (width 0.254) (layer "B.Cu") (net 3))
-  (segment (start 175.774999 119.625001) (end 177.450293 121.300295) (width 0.25) (layer "B.Cu") (net 3))
   (segment (start 147 100.6) (end 147 103.575) (width 0.254) (layer "B.Cu") (net 3))
   (segment (start 154.46 56) (end 157.46 53) (width 0.254) (layer "B.Cu") (net 3))
@@
   (segment (start 163.44 147.9) (end 171.459052 147.9) (width 0.254) (layer "B.Cu") (net 3))
   (segment (start 185.699705 139.033054) (end 185.699705 139.4332) (width 0.254) (layer "B.Cu") (net 3))
-  (segment (start 177.450293 121.300295) (end 201.9732 121.300295) (width 0.25) (layer "B.Cu") (net 3))
   (segment (start 191.437949 63.697157) (end 185.767592 58.0268) (width 0.254) (layer "B.Cu") (net 3))
   (segment (start 160.8 93.8) (end 160.8 98.8) (width 0.254) (layer "B.Cu") (net 3))
@@
   (segment (start 146.123148 56) (end 154.46 56) (width 0.254) (layer "B.Cu") (net 3))
   (segment (start 198.160408 74.300295) (end 191.437949 67.577836) (width 0.254) (layer "B.Cu") (net 3))
+  (segment (start 176.149998 120) (end 200.672905 120) (width 0.25) (layer "B.Cu") (net 3))
   (segment (start 145.382048 55.2589) (end 140.074148 60.5668) (width 0.254) (layer "B.Cu") (net 3))
   (segment (start 179.925852 139.4332) (end 185.699705 139.4332) (width 0.254) (layer "B.Cu") (net 3))
@@
   (segment (start 201.9732 113.793748) (end 201.9732 121.300295) (width 0.254) (layer "B.Cu") (net 3))
   (segment (start 138.699705 141.9732) (end 134.838828 141.9732) (width 0.254) (layer "B.Cu") (net 3))
+  (segment (start 200.672905 120) (end 201.9732 121.300295) (width 0.25) (layer "B.Cu") (net 3))
   (segment (start 200.700408 121.300295) (end 195.030051 126.970652) (width 0.254) (layer "B.Cu") (net 3))
   (segment (start 160.2 109.8) (end 168.4 101.6) (width 0.254) (layer "B.Cu") (net 3))
@@
   (segment (start 171.6 97.45) (end 172.88 98.73) (width 0.254) (layer "B.Cu") (net 15))
   (segment (start 172.6 80.8) (end 175 83.2) (width 0.254) (layer "B.Cu") (net 15))
-  (segment (start 160 95.2) (end 160 95.618766) (width 0.254) (layer "F.Cu") (net 24))
-  (segment (start 160 95.618766) (end 160.770403 96.389169) (width 0.254) (layer "F.Cu") (net 24))
+  (segment (start 166.6 90.925126) (end 161.705895 95.819231) (width 0.254) (layer "F.Cu") (net 24))
+  (segment (start 166.6 90.6) (end 166.6 90.925126) (width 0.254) (layer "F.Cu") (net 24))
   (segment (start 131.3 99.5) (end 132.6 98.2) (width 0.254) (layer "F.Cu") (net 24))
-  (segment (start 160.770403 96.389169) (end 161.135957 96.389169) (width 0.254) (layer "F.Cu") (net 24))
-  (segment (start 161.135957 96.389169) (end 161.705895 95.819231) (width 0.254) (layer "F.Cu") (net 24))
-  (segment (start 160 95.2) (end 160 91.4) (width 0.254) (layer "F.Cu") (net 24))
   (segment (start 128.6 99.5) (end 131.3 99.5) (width 0.254) (layer "F.Cu") (net 24))
   (via (at 132.6 98.2) (size 0.8) (drill 0.4) (layers "F.Cu" "B.Cu") (net 24))
-  (via (at 160 91.4) (size 0.8) (drill 0.4) (layers "F.Cu" "B.Cu") (net 24))
-  (segment (start 132.6 98.2) (end 139.4 91.4) (width 0.254) (layer "B.Cu") (net 24))
-  (segment (start 160 91.4) (end 139.4 91.4) (width 0.254) (layer "B.Cu") (net 24))
+  (via (at 166.6 90.6) (size 0.8) (drill 0.4) (layers "F.Cu" "B.Cu") (net 24))
+  (segment (start 166.6 90.6) (end 165.8 91.4) (width 0.254) (layer "B.Cu") (net 24))
+  (segment (start 139.4 91.4) (end 132.6 98.2) (width 0.254) (layer "B.Cu") (net 24))
+  (segment (start 165.8 91.4) (end 139.4 91.4) (width 0.254) (layer "B.Cu") (net 24))
   (segment (start 132.9 100.5) (end 134.2 99.2) (width 0.254) (layer "F.Cu") (net 25))
   (segment (start 159.001212 92.401212) (end 159 92.4) (width 0.254) (layer "F.Cu") (net 25))
