File: 2023l3-int-rounded.kicad_pcb (KiCad board)
At the start: 2 copper layers, 180.2 x 110 mm, 52 parts, among them IC1 STM32F103CBTx, J1 0526101433, J2 Conn_01x03_Pin, J3 Conn_01x04, SW1 SW_DIP_x02, SW2 SW_Push, SW3 SW_Push, U1 DEV-15583, U10 TSSP58038, U11 TSSP58038, U12 TSSP58038, U13 TSSP58038, U14 TSSP58038, U15 TSSP58038, U16 TSSP58038, U17 TSSP58038, U18 TSSP58038, U19 TSSP58038, U2 OpenMV H7, U20 TSSP58038, U21 TSSP58038, U22 TSSP58038, U23 TSSP58038, U24 TSSP58038, U25 TSSP58038, U26 TSSP58038, U27 TSSP58038, U28 xiao-esp32c3, U3 BNO085, U4 TSSP58038, U5 TSSP58038, U6 TSSP58038, U7 TSSP58038, U8 TSSP58038, U9 TSSP58038, Y1 8Mhz

Commit message: final
Routing:
- net /C TX: track 46.6 -> 48.5 mm
- net +3V3: track 495.9 -> 494.3 mm
