File: ir.kicad_sch (KiCad schematic)
At the start: 38 parts

Commit message: reee
Connections:
- net IR7: now also U?.27 (PB14); no longer U?.21 (PB10)
- no-connect marks 7 -> 6
Changed lines of the file:
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@@
   (no_connect (at 232.41 118.11))
   (no_connect (at 232.41 85.09))
-  (no_connect (at 232.41 125.73))
   (no_connect (at 232.41 123.19))
   (no_connect (at 245.11 57.15))
@@
     (stroke (width 0) (type default))
   )
+  (wire (pts (xy 226.06 125.73) (xy 232.41 125.73))
+    (stroke (width 0) (type default))
+  )
   (wire (pts (xy 135.89 36.83) (xy 143.51 36.83))
     (stroke (width 0) (type default))
@@
     (stroke (width 0) (type default))
   )
-  (wire (pts (xy 226.06 115.57) (xy 232.41 115.57))
-    (stroke (width 0) (type default))
-  )
   (wire (pts (xy 135.89 62.23) (xy 143.51 62.23))
     (stroke (width 0) (type default))
@@
     (effects (font (size 1.27 1.27)) (justify left bottom))
   )
+  (label "IR7" (at 227.33 125.73 0) (fields_autoplaced)
+    (effects (font (size 1.27 1.27)) (justify left bottom))
+  )
   (label "IR2" (at 97.79 36.83 0) (fields_autoplaced)
     (effects (font (size 1.27 1.27)) (justify left bottom))
@@
     (effects (font (size 1.27 1.27)) (justify right bottom))
   )
-  (label "IR7" (at 227.33 115.57 0) (fields_autoplaced)
-    (effects (font (size 1.27 1.27)) (justify left bottom))
-  )
   (label "IR16" (at 59.69 139.7 0) (fields_autoplaced)

Commit message: done
Parts:
- J?: footprint Connector_PinHeader_2.54mm:PinHeader_1x04_P2.54mm_Horizontal -> Connector_JST:JST_SH_SM04B-SRSS-TB_1x04-1MP_P1.00mm_Horizontal
Connections:
- net +3V3: now also J?.4 (Pin_4); no longer J?.1 (Pin_1)
- net GND: now also J?.1 (Pin_1); no longer J?.4 (Pin_4)
- net IR7: now also U?.28 (PB15); no longer U?.27 (PB14)
- net IR8: now also U?.27 (PB14); no longer U?.28 (PB15)
- net SWCLK: now also J?.3 (Pin_3); no longer J?.2 (Pin_2)
- net SWDIO: now also J?.2 (Pin_2); no longer J?.3 (Pin_3)
